Commit message: изменения описания робота

File: src/rob_box_description/urdf/rob_box.urdf (robot description, URDF)
Before this commit: robot rob_box, 7 links, 6 joints
Links:
- link base_link: geometry collision box size=0.4757 0.238 0.1885; visual box size=0.4757 0.238 0.1885
- link left_front_wheel: geometry collision cylinder length=0.05 radius=0.115; visual cylinder length=0.05 radius=0.115
- link left_rear_wheel: geometry collision cylinder length=0.05 radius=0.115; visual cylinder length=0.05 radius=0.115
- link left_rocker: geometry collision box size=0.28934 0.05 0.01; visual mesh filename=package://rob_box_description/meshes/rocker.stl scale=0.001 0.001 0.001
- link right_front_wheel: geometry collision cylinder length=0.05 radius=0.115; visual cylinder length=0.05 radius=0.115
- link right_rear_wheel: geometry collision cylinder length=0.05 radius=0.115; visual cylinder length=0.05 radius=0.115
- link right_rocker: geometry collision box size=0.28934 0.05 0.01; visual mesh filename=package://rob_box_description/meshes/rocker.stl scale=0.001 0.001 0.001
Joints:
- joint left_front_wheel_joint: origin xyz=0.25 0 -0.15 rpy=0 0 0 -> xyz=0.14467 0 -0.025 rpy=0 0 0
- joint left_rear_wheel_joint: origin xyz=-0.25 0 -0.15 rpy=0 0 0 -> xyz=-0.14467 0 -0.025 rpy=0 0 0
- joint left_rocker_joint: axis 0 0 1 -> 0 1 0; origin xyz=0 0.3 0.1 rpy=0 0 0 -> xyz=0 0.23048 0.09425 rpy=0 0 0
- joint right_front_wheel_joint: origin xyz=0.25 0 -0.15 rpy=0 0 0 -> xyz=0.14467 0 -0.025 rpy=0 0 0
- joint right_rear_wheel_joint: origin xyz=-0.25 0 -0.15 rpy=0 0 0 -> xyz=-0.14467 0 -0.025 rpy=0 0 0
- joint right_rocker_joint: axis 0 0 1 -> 0 1 0; origin xyz=0 -0.3 0.1 rpy=0 0 0 -> xyz=0 -0.23048 0.09425 rpy=0 0 0

Commit message: Добавил лидар и камеры

File: src/rob_box_description/urdf/rob_box.urdf (robot description, URDF)
Before this commit: robot rob_box, 7 links, 6 joints
Links:
- added link depth_camera, mass 0.2; collision box size=0.05 0.03 0.03; visual box size=0.05 0.03 0.03
- added link lidar, mass 0.5; collision cylinder length=0.1 radius=0.05; visual cylinder length=0.1 radius=0.05
- added link rgb_camera, mass 0.1; collision box size=0.05 0.03 0.03; visual box size=0.05 0.03 0.03
- link base_link: geometry collision box size=0.4757 0.238 0.1885; visual box size=0.4757 0.238 0.1885
- link left_front_wheel: geometry collision cylinder length=0.05 radius=0.115; visual mesh filename=package://rob_box_description/meshes/wheel.stl scale=0.001 0.001 0.001
- link left_rear_wheel: geometry collision cylinder length=0.05 radius=0.115; visual mesh filename=package://rob_box_description/meshes/wheel.stl scale=0.001 0.001 0.001
- link right_front_wheel: geometry collision cylinder length=0.05 radius=0.115; visual mesh filename=package://rob_box_description/meshes/wheel.stl scale=0.001 0.001 0.001
- link right_rear_wheel: geometry collision cylinder length=0.05 radius=0.115; visual mesh filename=package://rob_box_description/meshes/wheel.stl scale=0.001 0.001 0.001
- link right_rocker: geometry collision box size=0.28934 0.05 0.01; visual mesh filename=package://rob_box_description/meshes/rocker.stl scale=-0.001 0.001 0.001
Joints:
- added joint depth_camera_joint: type fixed, parent base_link, child depth_camera, origin xyz=0.2 0 0.1 rpy=0 0 0
- added joint lidar_joint: type fixed, parent base_link, child lidar, origin xyz=0 0 0.2 rpy=0 0 0
- added joint rgb_camera_joint: type fixed, parent base_link, child rgb_camera, origin xyz=-0.2 0 0.1 rpy=0 0 0
- joint left_front_wheel_joint: origin xyz=0.14467 0 -0.025 rpy=0 0 0 -> xyz=0.14467 0 -0.11 rpy=0 0 0
- joint left_rear_wheel_joint: origin xyz=-0.14467 0 -0.025 rpy=0 0 0 -> xyz=-0.14467 0 -0.11 rpy=0 0 0
- joint left_rocker_joint: origin xyz=0 0.23048 0.09425 rpy=0 0 0 -> xyz=0 0.18047999999999997 0.09425 rpy=0 0 0
- joint right_front_wheel_joint: origin xyz=0.14467 0 -0.025 rpy=0 0 0 -> xyz=0.14467 0 -0.11 rpy=0 0 0
- joint right_rear_wheel_joint: origin xyz=-0.14467 0 -0.025 rpy=0 0 0 -> xyz=-0.14467 0 -0.11 rpy=0 0 0
- joint right_rocker_joint: origin xyz=0 -0.23048 0.09425 rpy=0 0 0 -> xyz=0 -0.18047999999999997 0.09425 rpy=0 0 0

File: src/rob_box_description/urdf/rob_box.xacro (robot description, xacro)
@@ -25,5 +25,4 @@
 		<visual>
 			<origin xyz="0 -0.18 -0.02" rpy="0 0 -1.5708"/>
-			<!-- Позиция и ориентация меша -->
 			<geometry>
 				<mesh filename="package://rob_box_description/meshes/body_case.stl" scale="0.001 0.001 0.001"/>
@@ -31,5 +30,4 @@
 			<material name="silver">
 				<color rgba="0.75 0.75 0.75 1"/>
-				<!-- Серый цвет -->
 			</material>
 		</visual>
@@ -51,5 +49,4 @@
 			<visual>
 				<origin xyz="${-0.0035*side} 0 0.1451" rpy="1.5708 0 ${rotation_z}"/>
-				<!-- Поворот на 90 градусов вокруг X и Z -->
 				<geometry>
 					<mesh filename="package://rob_box_description/meshes/wheel.stl" scale="0.001 0.001 0.001"/>
@@ -57,10 +54,8 @@
 				<material name="black">
 					<color rgba="0 0 0 1"/>
-					<!-- Черный цвет -->
 				</material>
 			</visual>
 			<collision>
 				<origin xyz="0 ${0.05*side} 0" rpy="1.5708 0 0"/>
-				<!-- Поворот на 90 градусов вокруг оси X -->
 				<geometry>
 					<cylinder radius="${wheel_radius}" length="${wheel_length}"/>
@@ -78,5 +73,4 @@
 			<origin xyz="${origin_xyz}" rpy="0 0 0"/>
 			<axis xyz="0 1 0"/>
-			<!-- Ось вращения колеса -->
 		</joint>
 	</xacro:macro>
@@ -84,10 +78,9 @@
 		<link name="${name}">
 			<visual>
-				<origin xyz="0 0 -0.11" rpy="0 3.1416  -1.5708"/>
-				<!-- Поворот вокруг оси Z -->
+				<origin xyz="0 0 -0.11" rpy="0 3.1416 -1.5708"/>
 				<geometry>
 					<mesh filename="package://rob_box_description/meshes/rocker.stl" scale="${side * 0.001} 0.001 0.001"/>
 				</geometry>
-				<material name="black">
+				<material name="silver">
 					<color rgba="0.5 0.5 0.5 1"/>
 				</material>
@@ -110,5 +103,93 @@
 			<origin xyz="0 ${side * 0.23048 + side_x} 0.09425" rpy="0 0 0"/>
 			<axis xyz="0 1 0"/>
-			<limit effort="10" velocity="1" lower="-0.5" upper="0.5"/>
+			<limit effort="10" velocity="1" lower="-0.3" upper="0.3"/>
+		</joint>
+	</xacro:macro>
+	<!-- Сенсоры -->
+	<xacro:macro name="lidar" params="name parent_link origin_xyz">
+		<link name="${name}">
+			<visual>
+				<origin xyz="0 0 0" rpy="0 0 0"/>
+				<geometry>
+					<cylinder radius="0.05" length="0.1"/>
+				</geometry>
+				<material name="black">
+					<color rgba="0 0 0 1"/>
+				</material>
+			</visual>
+			<collision>
+				<origin xyz="0 0 0" rpy="0 0 0"/>
+				<geometry>
+					<cylinder radius="0.05" length="0.1"/>
+				</geometry>
+			</collision>
+			<inertial>
+				<mass value="0.5"/>
+				<origin xyz="0 0 0"/>
+				<inertia ixx="0.01" ixy="0" ixz="0" iyy="0.01" iyz="0" izz="0.01"/>
+			</inertial>
+		</link>
+		<joint name="${name}_joint" type="fixed">
+			<parent link="${parent_link}"/>
+			<child link="${name}"/>
+			<origin xyz="${origin_xyz}" rpy="0 0 0"/>
+		</joint>
+	</xacro:macro>
+	<xacro:macro name="depth_camera" params="name parent_link origin_xyz">
+		<link name="${name}">
+			<visual>
+				<origin xyz="0 0 0" rpy="0 0 0"/>
+				<geometry>
+					<box size="0.05 0.03 0.03"/>
+				</geometry>
+				<material name="gray">
+					<color rgba="0.5 0.5 0.5 1"/>
+				</material>
+			</visual>
+			<collision>
+				<origin xyz="0 0 0" rpy="0 0 0"/>
+				<geometry>
+					<box size="0.05 0.03 0.03"/>
+				</geometry>
+			</collision>
+			<inertial>
+				<mass value="0.2"/>
+				<origin xyz="0 0 0"/>
+				<inertia ixx="0.001" ixy="0" ixz="0" iyy="0.001" iyz="0" izz="0.001"/>
+			</inertial>
+		</link>
+		<joint name="${name}_joint" type="fixed">
+			<parent link="${parent_link}"/>
+			<child link="${name}"/>
+			<origin xyz="${origin_xyz}" rpy="0 0 0"/>
+		</joint>
+	</xacro:macro>
+	<xacro:macro name="rgb_camera" params="name parent_link origin_xyz">
+		<link name="${name}">
+			<visual>
+				<origin xyz="0 0 0" rpy="1.5708 0 0"/>
+				<geometry>
+					<box size="0.05 0.03 0.03"/>
+				</geometry>
+				<material name="blue">
+					<color rgba="0 0 1 1"/>
+				</material>
+			</visual>
+			<collision>
+				<origin xyz="0 0 0" rpy="1.5708 0 0"/>
+				<geometry>
+					<box size="0.05 0.03 0.03"/>
+				</geometry>
+			</collision>
+			<inertial>
+				<mass value="0.1"/>
+				<origin xyz="0 0 0"/>
+				<inertia ixx="0.001" ixy="0" ixz="0" iyy="0.001" iyz="0" izz="0.001"/>
+			</inertial>
+		</link>
+		<joint name="${name}_joint" type="fixed">
+			<parent link="${parent_link}"/>
+			<child link="${name}"/>
+			<origin xyz="${origin_xyz}" rpy="0 0 0"/>
 		</joint>
 	</xacro:macro>
@@ -116,8 +197,11 @@
 	<xacro:rocker name="left_rocker" side="1" side_x="-0.05"/>
 	<xacro:rocker name="right_rocker" side="-1" side_x="0.05"/>
-	<!-- Использование макросов -->
 	<xacro:wheel name="left_front_wheel" parent_link="left_rocker" origin_xyz="0.14467 0 -0.11" rotation_z="1.5708" side="1"/>
 	<xacro:wheel name="left_rear_wheel" parent_link="left_rocker" origin_xyz="-0.14467 0 -0.11" rotation_z="1.5708" side="1"/>
 	<xacro:wheel name="right_front_wheel" parent_link="right_rocker" origin_xyz="0.14467 0 -0.11" rotation_z="-1.5708" side="-1"/>
 	<xacro:wheel name="right_rear_wheel" parent_link="right_rocker" origin_xyz="-0.14467 0 -0.11" rotation_z="-1.5708" side="-1"/>
+	<!-- Сенсоры -->
+	<xacro:lidar name="lidar" parent_link="base_link" origin_xyz="0.2 0 0.2"/>
+	<xacro:depth_camera name="depth_camera" parent_link="base_link" origin_xyz="0.2 0 0.3"/>
+	<xacro:rgb_camera name="rgb_camera" parent_link="base_link" origin_xyz="-0.2 0 0.2"/>
 </robot>

Commit message: lidar&cameras

File: src/rob_box_description/urdf/rob_box.urdf (robot description, URDF)
Before this commit: robot rob_box, 10 links, 9 joints
Links:
- link depth_camera: geometry collision box size=0.0175 0.091 0.028; visual box size=0.0175 0.091 0.028
- link lidar: mass 0.5 -> 0.06; geometry collision cylinder length=0.0361 radius=0.026; visual cylinder length=0.0361 radius=0.026
Joints:
- joint depth_camera_joint: origin xyz=0.2 0 0.1 rpy=0 0 0 -> xyz=0.29 0 0.167 rpy=0 0 0
- joint left_rocker_joint: limit lower=-0.5 upper=0.5 effort=10 velocity=1 -> lower=-0.3 upper=0.3 effort=10 velocity=1
- joint lidar_joint: origin xyz=0 0 0.2 rpy=0 0 0 -> xyz=0.25 0 0.2 rpy=0 0 0
- joint rgb_camera_joint: origin xyz=-0.2 0 0.1 rpy=0 0 0 -> xyz=0.25 0.2 0.167 rpy=0 0 0
- joint right_rocker_joint: limit lower=-0.5 upper=0.5 effort=10 velocity=1 -> lower=-0.3 upper=0.3 effort=10 velocity=1

File: src/rob_box_description/urdf/rob_box.xacro (robot description, xacro)
@@ -112,5 +112,5 @@
 				<origin xyz="0 0 0" rpy="0 0 0"/>
 				<geometry>
-					<cylinder radius="0.05" length="0.1"/>
+					<cylinder radius="0.026" length="0.0361"/>
 				</geometry>
 				<material name="black">
@@ -121,11 +121,11 @@
 				<origin xyz="0 0 0" rpy="0 0 0"/>
 				<geometry>
-					<cylinder radius="0.05" length="0.1"/>
-				</geometry>
-			</collision>
-			<inertial>
-				<mass value="0.5"/>
-				<origin xyz="0 0 0"/>
-				<inertia ixx="0.01" ixy="0" ixz="0" iyy="0.01" iyz="0" izz="0.01"/>
+					<cylinder radius="0.026" length="0.0361"/>
+				</geometry>
+			</collision>
+			<inertial>
+				<mass value="0.06"/>
+				<origin xyz="0 0 0"/>
+				<inertia ixx="0.0001" ixy="0" ixz="0" iyy="0.0001" iyz="0" izz="0.0001"/>
 			</inertial>
 		</link>
@@ -141,5 +141,5 @@
 				<origin xyz="0 0 0" rpy="0 0 0"/>
 				<geometry>
-					<box size="0.05 0.03 0.03"/>
+					<box size="0.0175 0.091 0.028"/>
 				</geometry>
 				<material name="gray">
@@ -150,5 +150,5 @@
 				<origin xyz="0 0 0" rpy="0 0 0"/>
 				<geometry>
-					<box size="0.05 0.03 0.03"/>
+					<box size="0.0175 0.091 0.028"/>
 				</geometry>
 			</collision>
@@ -156,5 +156,5 @@
 				<mass value="0.2"/>
 				<origin xyz="0 0 0"/>
-				<inertia ixx="0.001" ixy="0" ixz="0" iyy="0.001" iyz="0" izz="0.001"/>
+				<inertia ixx="0.0001" ixy="0" ixz="0" iyy="0.0001" iyz="0" izz="0.0001"/>
 			</inertial>
 		</link>
@@ -185,5 +185,5 @@
 				<mass value="0.1"/>
 				<origin xyz="0 0 0"/>
-				<inertia ixx="0.001" ixy="0" ixz="0" iyy="0.001" iyz="0" izz="0.001"/>
+				<inertia ixx="0.0001" ixy="0" ixz="0" iyy="0.0001" iyz="0" izz="0.0001"/>
 			</inertial>
 		</link>
@@ -202,6 +202,6 @@
 	<xacro:wheel name="right_rear_wheel" parent_link="right_rocker" origin_xyz="-0.14467 0 -0.11" rotation_z="-1.5708" side="-1"/>
 	<!-- Сенсоры -->
-	<xacro:lidar name="lidar" parent_link="base_link" origin_xyz="0.2 0 0.2"/>
-	<xacro:depth_camera name="depth_camera" parent_link="base_link" origin_xyz="0.2 0 0.3"/>
-	<xacro:rgb_camera name="rgb_camera" parent_link="base_link" origin_xyz="-0.2 0 0.2"/>
+	<xacro:lidar name="lidar" parent_link="base_link" origin_xyz="0.25 0 0.2"/>
+	<xacro:depth_camera name="depth_camera" parent_link="base_link" origin_xyz="0.29 0 0.167"/>
+	<xacro:rgb_camera name="rgb_camera" parent_link="base_link" origin_xyz="0.25 0.2 0.167"/>
 </robot>

Commit message: починил качение рокера

File: src/rob_box_description/urdf/rob_box.urdf (robot description, URDF)
Before this commit: robot rob_box, 10 links, 9 joints
Joints:
- joint left_rocker_joint: type revolute -> fixed
- joint right_rocker_joint: type revolute -> fixed

File: src/rob_box_description/urdf/rob_box.xacro (robot description, xacro)
@@ -98,5 +98,5 @@
 			</inertial>
 		</link>
-		<joint name="${name}_joint" type="revolute">
+		<joint name="${name}_joint" type="fixed">
 			<parent link="base_link"/>
 			<child link="${name}"/>

Commit message: robot definition

File: src/rob_box_description/urdf/rob_box.urdf (robot description, URDF)
Before this commit: robot rob_box, 10 links, 9 joints
Links:
- removed link depth_camera
- removed link lidar
- added link lslidar_n10, mass 0.06; collision cylinder length=0.0361 radius=0.026; visual cylinder length=0.0361 radius=0.026
Joints:
- removed joint depth_camera_joint
- removed joint lidar_joint
- added joint lslidar_n10_joint: type fixed, parent base_link, child lslidar_n10, origin xyz=0.25 0 0.2 rpy=0 0 0

File: src/rob_box_description/urdf/rob_box.xacro (robot description, xacro)
@@ -107,5 +107,5 @@
 	</xacro:macro>
 	<!-- Сенсоры -->
-	<xacro:macro name="lidar" params="name parent_link origin_xyz">
+	<xacro:macro name="lidar" params="name parent_link origin_xyz topic_name">
 		<link name="${name}">
 			<visual>
@@ -135,24 +135,57 @@
 			<origin xyz="${origin_xyz}" rpy="0 0 0"/>
 		</joint>
-	</xacro:macro>
-	<xacro:macro name="depth_camera" params="name parent_link origin_xyz">
-		<link name="${name}">
-			<visual>
-				<origin xyz="0 0 0" rpy="0 0 0"/>
-				<geometry>
-					<box size="0.0175 0.091 0.028"/>
-				</geometry>
-				<material name="gray">
-					<color rgba="0.5 0.5 0.5 1"/>
-				</material>
-			</visual>
-			<collision>
-				<origin xyz="0 0 0" rpy="0 0 0"/>
-				<geometry>
-					<box size="0.0175 0.091 0.028"/>
-				</geometry>
-			</collision>
-			<inertial>
-				<mass value="0.2"/>
+		<gazebo reference="${name}">
+			<sensor name="${name}_sensor" type="gpu_lidar">
+				<pose>0 0 0 0 0 0</pose>
+				<topic>${topic_name}</topic>
+				<update_rate>10</update_rate>
+				<ray>
+					<scan>
+						<horizontal>
+							<samples>640</samples>
+							<resolution>1</resolution>
+							<min_angle>-1.396263</min_angle>
+							<max_angle>1.396263</max_angle>
+						</horizontal>
+						<vertical>
+							<samples>1</samples>
+							<resolution>0.01</resolution>
+							<min_angle>0</min_angle>
+							<max_angle>0</max_angle>
+						</vertical>
+					</scan>
+					<range>
+						<min>0.08</min>
+						<max>10.0</max>
+						<resolution>0.01</resolution>
+					</range>
+				</ray>
+				<always_on>1</always_on>
+				<visualize>true</visualize>
+			</sensor>
+			<plugin filename="libignition-gazebo-sensors-system.so" name="ignition::gazebo::systems::Sensors">
+				<render_engine>ogre2</render_engine>
+			</plugin>
+		</gazebo>
+	</xacro:macro>
+	<xacro:macro name="rgb_camera" params="name parent_link origin_xyz topic_name">
+		<link name="${name}">
+			<visual>
+				<origin xyz="0 0 0" rpy="1.5708 0 0"/>
+				<geometry>
+					<box size="0.05 0.03 0.03"/>
+				</geometry>
+				<material name="blue">
+					<color rgba="0 0 1 1"/>
+				</material>
+			</visual>
+			<collision>
+				<origin xyz="0 0 0" rpy="1.5708 0 0"/>
+				<geometry>
+					<box size="0.05 0.03 0.03"/>
+				</geometry>
+			</collision>
+			<inertial>
+				<mass value="0.1"/>
 				<origin xyz="0 0 0"/>
 				<inertia ixx="0.0001" ixy="0" ixz="0" iyy="0.0001" iyz="0" izz="0.0001"/>
@@ -164,33 +197,26 @@
 			<origin xyz="${origin_xyz}" rpy="0 0 0"/>
 		</joint>
-	</xacro:macro>
-	<xacro:macro name="rgb_camera" params="name parent_link origin_xyz">
-		<link name="${name}">
-			<visual>
-				<origin xyz="0 0 0" rpy="1.5708 0 0"/>
-				<geometry>
-					<box size="0.05 0.03 0.03"/>
-				</geometry>
-				<material name="blue">
-					<color rgba="0 0 1 1"/>
-				</material>
-			</visual>
-			<collision>
-				<origin xyz="0 0 0" rpy="1.5708 0 0"/>
-				<geometry>
-					<box size="0.05 0.03 0.03"/>
-				</geometry>
-			</collision>
-			<inertial>
-				<mass value="0.1"/>
-				<origin xyz="0 0 0"/>
-				<inertia ixx="0.0001" ixy="0" ixz="0" iyy="0.0001" iyz="0" izz="0.0001"/>
-			</inertial>
-		</link>
-		<joint name="${name}_joint" type="fixed">
-			<parent link="${parent_link}"/>
-			<child link="${name}"/>
-			<origin xyz="${origin_xyz}" rpy="0 0 0"/>
-		</joint>
+		<gazebo reference="${name}">
+			<sensor name="${name}_sensor" type="camera">
+				<camera>
+					<horizontal_fov>1.047</horizontal_fov>
+					<image>
+						<width>640</width>
+						<height>480</height>
+					</image>
+					<clip>
+						<near>0.1</near>
+						<far>100</far>
+					</clip>
+				</camera>
+				<topic>${topic_name}</topic>
+				<update_rate>30</update_rate>
+				<always_on>1</always_on>
+				<visualize>true</visualize>
+			</sensor>
+			<plugin filename="libignition-gazebo-sensors-system.so" name="ignition::gazebo::systems::Sensors">
+				<render_engine>ogre2</render_engine>
+			</plugin>
+		</gazebo>
 	</xacro:macro>
 	<!-- Использование макросов -->
@@ -202,6 +228,5 @@
 	<xacro:wheel name="right_rear_wheel" parent_link="right_rocker" origin_xyz="-0.14467 0 -0.11" rotation_z="-1.5708" side="-1"/>
 	<!-- Сенсоры -->
-	<xacro:lidar name="lidar" parent_link="base_link" origin_xyz="0.25 0 0.2"/>
-	<xacro:depth_camera name="depth_camera" parent_link="base_link" origin_xyz="0.29 0 0.167"/>
-	<xacro:rgb_camera name="rgb_camera" parent_link="base_link" origin_xyz="0.25 0.2 0.167"/>
+	<xacro:lidar name="lslidar_n10" parent_link="base_link" origin_xyz="0.25 0 0.2" topic_name="/scan"/>
+	<xacro:rgb_camera name="rgb_camera" parent_link="base_link" origin_xyz="0.25 0.2 0.167" topic_name="/camera/image_raw"/>
 </robot>
