Commit message: fix(ros2_control): rename wheel joints to match controller_manager
- front_left_wheel_joint → left_front_wheel_joint
- rear_left_wheel_joint → left_rear_wheel_joint
- front_right_wheel_joint → right_front_wheel_joint
- rear_right_wheel_joint → right_rear_wheel_joint

Unified naming: left/right_front/rear_wheel across all configs

File: src/rob_box_description/urdf/rob_box_ros2_control.xacro (robot description, xacro)
@@ -19,7 +19,7 @@
     </hardware>
     <!-- ═══════════════════════════════════════════════════════════════ -->
-    <!-- Front Left Wheel -->
+    <!-- Left Front Wheel -->
     <!-- ═══════════════════════════════════════════════════════════════ -->
-    <joint name="front_left_wheel_joint">
+    <joint name="left_front_wheel_joint">
       <command_interface name="velocity">
         <param name="min">-10</param>  <!-- м/с -->
@@ -35,7 +35,7 @@
     </joint>
     <!-- ═══════════════════════════════════════════════════════════════ -->
-    <!-- Front Right Wheel -->
+    <!-- Right Front Wheel -->
     <!-- ═══════════════════════════════════════════════════════════════ -->
-    <joint name="front_right_wheel_joint">
+    <joint name="right_front_wheel_joint">
       <command_interface name="velocity">
         <param name="min">-10</param>
@@ -50,7 +50,7 @@
     </joint>
     <!-- ═══════════════════════════════════════════════════════════════ -->
-    <!-- Rear Left Wheel -->
+    <!-- Left Rear Wheel -->
     <!-- ═══════════════════════════════════════════════════════════════ -->
-    <joint name="rear_left_wheel_joint">
+    <joint name="left_rear_wheel_joint">
       <command_interface name="velocity">
         <param name="min">-10</param>
@@ -65,7 +65,7 @@
     </joint>
     <!-- ═══════════════════════════════════════════════════════════════ -->
-    <!-- Rear Right Wheel -->
+    <!-- Right Rear Wheel -->
     <!-- ═══════════════════════════════════════════════════════════════ -->
-    <joint name="rear_right_wheel_joint">
+    <joint name="right_rear_wheel_joint">
       <command_interface name="velocity">
         <param name="min">-10</param>
