Commit message: Add robot_state_publisher and fix TF tree
URDF changes:
- Created oak_d_camera macro with proper frame hierarchy
- Replaced simple rgb_camera with OAK-D-Lite model (61g, proper dimensions)
- Frame chain: base_link  camera_link  camera  camera_color_optical_frame
- Added depth frames: camera_depth_frame, camera_depth_optical_frame

Docker changes:
- New container: robot-state-publisher on Main Pi
- Publishes complete TF tree from URDF for all nodes
- Read-only mount of /src for URDF access

Camera config:
- i_publish_tf_from_calibration: false (TF from robot_state_publisher)
- i_tf_base_frame: camera_link (not base_link)
- Camera no longer publishes conflicting TF

This fixes RTAB-Map error:
'base_link_color_optical_frame does not exist'

Now robot_state_publisher provides complete transform chain,
RTAB-Map can lookup base_link  camera_color_optical_frame.

File: src/rob_box_description/urdf/rob_box.xacro (robot description, xacro)
@@ -169,54 +169,78 @@
 		</gazebo>
 	</xacro:macro>
-	<xacro:macro name="rgb_camera" params="name parent_link origin_xyz topic_name">
-		<link name="${name}">
-			<visual>
-				<origin xyz="0 0 0" rpy="1.5708 0 0"/>
-				<geometry>
-					<box size="0.05 0.03 0.03"/>
-				</geometry>
-				<material name="blue">
-					<color rgba="0 0 1 1"/>
-				</material>
-			</visual>
-			<collision>
-				<origin xyz="0 0 0" rpy="1.5708 0 0"/>
-				<geometry>
-					<box size="0.05 0.03 0.03"/>
-				</geometry>
-			</collision>
-			<inertial>
-				<mass value="0.1"/>
-				<origin xyz="0 0 0"/>
-				<inertia ixx="0.0001" ixy="0" ixz="0" iyy="0.0001" iyz="0" izz="0.0001"/>
-			</inertial>
-		</link>
+	<!-- OAK-D Camera Macro - соответствует реальной структуре фреймов depthai_ros_driver -->
+	<xacro:macro name="oak_d_camera" params="name parent_link origin_xyz origin_rpy">
+		<!-- camera_link - основной корпус камеры -->
+		<link name="${name}_link">
+			<visual>
+				<origin xyz="0 0 0" rpy="0 0 0"/>
+				<geometry>
+					<box size="0.097 0.0275 0.0214"/>  <!-- Размеры OAK-D-Lite -->
+				</geometry>
+				<material name="dark_grey">
+					<color rgba="0.2 0.2 0.2 1"/>
+				</material>
+			</visual>
+			<collision>
+				<origin xyz="0 0 0" rpy="0 0 0"/>
+				<geometry>
+					<box size="0.097 0.0275 0.0214"/>
+				</geometry>
+			</collision>
+			<inertial>
+				<mass value="0.061"/>  <!-- 61g вес OAK-D-Lite -->
+				<origin xyz="0 0 0"/>
+				<inertia ixx="0.00001" ixy="0" ixz="0" iyy="0.00001" iyz="0" izz="0.00001"/>
+			</inertial>
+		</link>
+		<!-- Присоединение к роботу -->
 		<joint name="${name}_joint" type="fixed">
 			<parent link="${parent_link}"/>
-			<child link="${name}"/>
-			<origin xyz="${origin_xyz}" rpy="0 0 0"/>
-		</joint>
-		<gazebo reference="${name}">
-			<sensor name="${name}_sensor" type="camera">
-				<camera>
-					<horizontal_fov>1.047</horizontal_fov>
-					<image>
-						<width>640</width>
-						<height>480</height>
-					</image>
-					<clip>
-						<near>0.1</near>
-						<far>100</far>
-					</clip>
-				</camera>
-				<topic>${topic_name}</topic>
-				<update_rate>30</update_rate>
-				<always_on>1</always_on>
-				<visualize>true</visualize>
-			</sensor>
-			<plugin filename="libignition-gazebo-sensors-system.so" name="ignition::gazebo::systems::Sensors">
-				<render_engine>ogre2</render_engine>
-			</plugin>
-		</gazebo>
+			<child link="${name}_link"/>
+			<origin xyz="${origin_xyz}" rpy="${origin_rpy}"/>
+		</joint>
+		<!-- camera (intermediate frame - используется depthai_ros_driver) -->
+		<link name="${name}"/>
+		<joint name="${name}_base_joint" type="fixed">
+			<parent link="${name}_link"/>
+			<child link="${name}"/>
+			<origin xyz="0 0 0" rpy="0 0 0"/>
+		</joint>
+		<!-- Color camera frames -->
+		<link name="${name}_color_frame"/>
+		<joint name="${name}_color_frame_joint" type="fixed">
+			<parent link="${name}"/>
+			<child link="${name}_color_frame"/>
+			<!-- Смещение RGB камеры относительно базы (из calibration) -->
+			<origin xyz="0 0 0" rpy="0 0 0"/>
+		</joint>
+		<link name="${name}_color_optical_frame"/>
+		<joint name="${name}_color_optical_frame_joint" type="fixed">
+			<parent link="${name}_color_frame"/>
+			<child link="${name}_color_optical_frame"/>
+			<!-- Optical frame: X right, Y down, Z forward (ROS camera convention) -->
+			<origin xyz="0 0 0" rpy="-1.5708 0 -1.5708"/>
+		</joint>
+		<!-- Depth/Stereo camera frames -->
+		<link name="${name}_depth_frame"/>
+		<joint name="${name}_depth_frame_joint" type="fixed">
+			<parent link="${name}"/>
+			<child link="${name}_depth_frame"/>
+			<!-- Depth камера немного смещена (левая камера stereo пары) -->
+			<origin xyz="0 0.0375 0" rpy="0 0 0"/>
+		</joint>
+		<link name="${name}_depth_optical_frame"/>
+		<joint name="${name}_depth_optical_frame_joint" type="fixed">
+			<parent link="${name}_depth_frame"/>
+			<child link="${name}_depth_optical_frame"/>
+			<origin xyz="0 0 0" rpy="-1.5708 0 -1.5708"/>
+		</joint>
+		<!-- IMU frame (если используется) -->
+		<link name="${name}_imu_frame"/>
+		<joint name="${name}_imu_frame_joint" type="fixed">
+			<parent link="${name}"/>
+			<child link="${name}_imu_frame"/>
+			<origin xyz="0 0 0" rpy="0 0 0"/>
+		</joint>
 	</xacro:macro>
 	<!-- Использование макросов -->
@@ -229,4 +253,5 @@
 	<!-- Сенсоры -->
 	<xacro:lidar name="lslidar_n10" parent_link="base_link" origin_xyz="0.25 0 0.2" topic_name="/scan"/>
-	<xacro:rgb_camera name="rgb_camera" parent_link="base_link" origin_xyz="0.25 0.2 0.167" topic_name="/camera/image_raw"/>
+	<!-- OAK-D-Lite камера на передней части робота -->
+	<xacro:oak_d_camera name="camera" parent_link="base_link" origin_xyz="0.25 0 0.167" origin_rpy="0 0 0"/>
 </robot>

Commit message: fix(urdf): добавить ros2_control секцию в rob_box.xacro, исправить имена джойнтов

File: src/rob_box_description/urdf/rob_box.xacro (robot description, xacro)
@@ -255,3 +255,5 @@
 	<!-- OAK-D-Lite камера на передней части робота -->
 	<xacro:oak_d_camera name="camera" parent_link="base_link" origin_xyz="0.25 0 0.167" origin_rpy="0 0 0"/>
+	<!-- ros2_control Hardware Interface - VESC Nexus -->
+	<xacro:include filename="$(find rob_box_description)/urdf/rob_box_ros2_control.xacro"/>
 </robot>

File: src/rob_box_description/urdf/rob_box_ros2_control.xacro (robot description, xacro)
@@ -19,7 +19,7 @@
     </hardware>
     <!-- ═══════════════════════════════════════════════════════════════ -->
-    <!-- Front Left Wheel -->
+    <!-- Left Front Wheel -->
     <!-- ═══════════════════════════════════════════════════════════════ -->
-    <joint name="front_left_wheel_joint">
+    <joint name="left_front_wheel_joint">
       <command_interface name="velocity">
         <param name="min">-10</param>  <!-- м/с -->
@@ -35,7 +35,7 @@
     </joint>
     <!-- ═══════════════════════════════════════════════════════════════ -->
-    <!-- Front Right Wheel -->
+    <!-- Right Front Wheel -->
     <!-- ═══════════════════════════════════════════════════════════════ -->
-    <joint name="front_right_wheel_joint">
+    <joint name="right_front_wheel_joint">
       <command_interface name="velocity">
         <param name="min">-10</param>
@@ -50,7 +50,7 @@
     </joint>
     <!-- ═══════════════════════════════════════════════════════════════ -->
-    <!-- Rear Left Wheel -->
+    <!-- Left Rear Wheel -->
     <!-- ═══════════════════════════════════════════════════════════════ -->
-    <joint name="rear_left_wheel_joint">
+    <joint name="left_rear_wheel_joint">
       <command_interface name="velocity">
         <param name="min">-10</param>
@@ -65,7 +65,7 @@
     </joint>
     <!-- ═══════════════════════════════════════════════════════════════ -->
-    <!-- Rear Right Wheel -->
+    <!-- Right Rear Wheel -->
     <!-- ═══════════════════════════════════════════════════════════════ -->
-    <joint name="rear_right_wheel_joint">
+    <joint name="right_rear_wheel_joint">
       <command_interface name="velocity">
         <param name="min">-10</param>

Commit message: fix(urdf): убрать placeholder box из base_link
- Удален белый box visual элемент (placeholder)
- Оставлен только mesh body_case.stl
- Исправлен визуальный баг (белый квадрат поверх модели)
- Проверено: lslidar_n10 frame генерируется корректно

File: src/rob_box_description/urdf/rob_box.xacro (robot description, xacro)
@@ -13,13 +13,4 @@
 	<!-- Основное шасси -->
 	<link name="base_link">
-		<visual>
-			<origin xyz="0 0 0.0565" rpy="0 0 0"/>
-			<geometry>
-				<box size="${base_size}"/>
-			</geometry>
-			<material name="white">
-				<color rgba="1 1 1 1"/>
-			</material>
-		</visual>
 		<!-- Меш body_case.stl -->
 		<visual>

Commit message: Add ceiling camera support with AprilTag detection
- Add ceiling-camera Dockerfile in docker/vision/ceiling-camera/
- Add ceiling-camera service to docker/vision/docker-compose.yaml
- Create camera config in docker/vision/config/ceiling-camera/camera_params.yaml
- Create startup script in docker/vision/scripts/ceiling-camera/start_ceiling_camera.sh
- Add usb_camera macro and ceiling_camera instance to URDF (rob_box.xacro)
- Update GitHub Actions workflow to build ceiling-camera image

Technical specs:
- 720p @ 10 Hz with YUY2 format
- JPEG compression at quality 85
- Zenoh middleware for Main Pi communication
- Proper TF frames (ceiling_camera_optical_frame)
- Following DOCKER_STANDARDS.md - configs/scripts mounted via volumes

Co-authored-by: GOODWORKRINKZ <237234482+GOODWORKRINKZ@users.noreply.github.com>

File: src/rob_box_description/urdf/rob_box.xacro (robot description, xacro)
@@ -235,4 +235,43 @@
 		</joint>
 	</xacro:macro>
+	<!-- Simple USB Camera Macro - для обычных USB камер (ceiling camera, etc.) -->
+	<xacro:macro name="usb_camera" params="name parent_link origin_xyz origin_rpy">
+		<!-- camera_link - основной корпус камеры -->
+		<link name="${name}_link">
+			<visual>
+				<origin xyz="0 0 0" rpy="0 0 0"/>
+				<geometry>
+					<box size="0.03 0.03 0.02"/>  <!-- Размеры generic USB камеры -->
+				</geometry>
+				<material name="black">
+					<color rgba="0.1 0.1 0.1 1"/>
+				</material>
+			</visual>
+			<collision>
+				<origin xyz="0 0 0" rpy="0 0 0"/>
+				<geometry>
+					<box size="0.03 0.03 0.02"/>
+				</geometry>
+			</collision>
+			<inertial>
+				<mass value="0.05"/>  <!-- ~50g -->
+				<origin xyz="0 0 0"/>
+				<inertia ixx="0.00001" ixy="0" ixz="0" iyy="0.00001" iyz="0" izz="0.00001"/>
+			</inertial>
+		</link>
+		<!-- Присоединение к роботу -->
+		<joint name="${name}_joint" type="fixed">
+			<parent link="${parent_link}"/>
+			<child link="${name}_link"/>
+			<origin xyz="${origin_xyz}" rpy="${origin_rpy}"/>
+		</joint>
+		<!-- Optical frame: X right, Y down, Z forward (ROS camera convention) -->
+		<link name="${name}_optical_frame"/>
+		<joint name="${name}_optical_frame_joint" type="fixed">
+			<parent link="${name}_link"/>
+			<child link="${name}_optical_frame"/>
+			<origin xyz="0 0 0" rpy="-1.5708 0 -1.5708"/>
+		</joint>
+	</xacro:macro>
 	<!-- Использование макросов -->
 	<xacro:rocker name="left_rocker" side="1" side_x="-0.05"/>
@@ -246,4 +285,6 @@
 	<!-- OAK-D-Lite камера на передней части робота -->
 	<xacro:oak_d_camera name="camera" parent_link="base_link" origin_xyz="0.25 0 0.167" origin_rpy="0 0 0"/>
+	<!-- Потолочная USB камера (направлена вертикально вверх) -->
+	<xacro:usb_camera name="ceiling_camera" parent_link="base_link" origin_xyz="0.0 0.0 0.25" origin_rpy="0 3.14159 0"/>
 	<!-- ros2_control Hardware Interface - VESC Nexus -->
 	<xacro:include filename="rob_box_ros2_control.xacro"/>

Commit message: fix: align camera frame names with depthai_ros_driver convention
- Update URDF to use camera_rgb_camera_optical_frame instead of camera_color_optical_frame
- Update URDF to use camera_stereo_camera_optical_frame instead of camera_depth_optical_frame
- Fix AprilTag topic remapping to subscribe to correct camera topics
- This resolves TF transform error between camera and base_link

Co-authored-by: GOODWORKRINKZ <237234482+GOODWORKRINKZ@users.noreply.github.com>

File: src/rob_box_description/urdf/rob_box.xacro (robot description, xacro)
@@ -198,31 +198,31 @@
 			<origin xyz="0 0 0" rpy="0 0 0"/>
 		</joint>
-		<!-- Color camera frames -->
-		<link name="${name}_color_frame"/>
-		<joint name="${name}_color_frame_joint" type="fixed">
+		<!-- RGB camera frames (depthai_ros_driver использует именование rgb_camera, не color) -->
+		<link name="${name}_rgb_camera_frame"/>
+		<joint name="${name}_rgb_camera_frame_joint" type="fixed">
 			<parent link="${name}"/>
-			<child link="${name}_color_frame"/>
+			<child link="${name}_rgb_camera_frame"/>
 			<!-- Смещение RGB камеры относительно базы (из calibration) -->
 			<origin xyz="0 0 0" rpy="0 0 0"/>
 		</joint>
-		<link name="${name}_color_optical_frame"/>
-		<joint name="${name}_color_optical_frame_joint" type="fixed">
-			<parent link="${name}_color_frame"/>
-			<child link="${name}_color_optical_frame"/>
+		<link name="${name}_rgb_camera_optical_frame"/>
+		<joint name="${name}_rgb_camera_optical_frame_joint" type="fixed">
+			<parent link="${name}_rgb_camera_frame"/>
+			<child link="${name}_rgb_camera_optical_frame"/>
 			<!-- Optical frame: X right, Y down, Z forward (ROS camera convention) -->
 			<origin xyz="0 0 0" rpy="-1.5708 0 -1.5708"/>
 		</joint>
 		<!-- Depth/Stereo camera frames -->
-		<link name="${name}_depth_frame"/>
-		<joint name="${name}_depth_frame_joint" type="fixed">
+		<link name="${name}_stereo_camera_frame"/>
+		<joint name="${name}_stereo_camera_frame_joint" type="fixed">
 			<parent link="${name}"/>
-			<child link="${name}_depth_frame"/>
+			<child link="${name}_stereo_camera_frame"/>
 			<!-- Depth камера немного смещена (левая камера stereo пары) -->
 			<origin xyz="0 0.0375 0" rpy="0 0 0"/>
 		</joint>
-		<link name="${name}_depth_optical_frame"/>
-		<joint name="${name}_depth_optical_frame_joint" type="fixed">
-			<parent link="${name}_depth_frame"/>
-			<child link="${name}_depth_optical_frame"/>
+		<link name="${name}_stereo_camera_optical_frame"/>
+		<joint name="${name}_stereo_camera_optical_frame_joint" type="fixed">
+			<parent link="${name}_stereo_camera_frame"/>
+			<child link="${name}_stereo_camera_optical_frame"/>
 			<origin xyz="0 0 0" rpy="-1.5708 0 -1.5708"/>
 		</joint>

Commit message: feat(urdf): update base_link and meshes from Fusion 360 export
Co-authored-by: GOODWORKRINKZ <237234482+GOODWORKRINKZ@users.noreply.github.com>

File: src/rob_box_description/urdf/rob_box.xacro (robot description, xacro)
@@ -1,6 +1,6 @@
 <?xml version="1.0"?>
 <robot name="rob_box" xmlns:xacro="http://www.ros.org/wiki/xacro">
-	<!-- Переменные -->
-	<xacro:property name="base_size" value="0.4757 0.238 0.1885"/>
+	<!-- Переменные - обновлено из Fusion 360 Export -->
+	<xacro:property name="base_size" value="0.4757 0.238 0.1885"/>  <!-- Legacy collision box, use mesh instead -->
 	<xacro:property name="wheel_radius" value="0.115"/>
 	<xacro:property name="wheel_length" value="0.05"/>
@@ -8,14 +8,21 @@
 	<xacro:property name="rocker_width" value="0.05"/>
 	<xacro:property name="rocker_thickness" value="0.01"/>
-	<xacro:property name="wheel_mass" value="2"/>
+	<xacro:property name="wheel_mass" value="21.68159743475603"/>  <!-- От Fusion 360: 21.68 кг -->
 	<xacro:property name="rocker_mass" value="3"/>
-	<xacro:property name="base_mass" value="10"/>
-	<!-- Основное шасси -->
+	<xacro:property name="base_mass" value="62.64527022934752"/>  <!-- От Fusion 360: 62.65 кг -->
+	<!-- Основное шасси - обновлено из Fusion 360 Export -->
 	<link name="base_link">
-		<!-- Меш body_case.stl -->
+		<!-- Меш base_link.stl из Fusion 360 - нормализован относительно base_link (0,0,0) -->
+		<inertial>
+			<!-- Инерциальные параметры из Fusion 360 -->
+			<origin xyz="-2.4090750286344156e-05 0.025488169162562517 0.14529190576177464" rpy="0 0 0"/>
+			<mass value="${base_mass}"/>
+			<inertia ixx="2.829827" iyy="1.926172" izz="3.653023" ixy="-0.001791" iyz="-0.302171" ixz="-0.001655"/>
+		</inertial>
 		<visual>
-			<origin xyz="0 -0.18 -0.02" rpy="0 0 -1.5708"/>
+			<!-- Меш без offset - base_link в (0,0,0) как требуется -->
+			<origin xyz="0 0 0" rpy="0 0 0"/>
 			<geometry>
-				<mesh filename="package://rob_box_description/meshes/body_case.stl" scale="0.001 0.001 0.001"/>
+				<mesh filename="package://rob_box_description/meshes/base_link.stl" scale="0.001 0.001 0.001"/>
 			</geometry>
 			<material name="silver">
@@ -24,14 +31,10 @@
 		</visual>
 		<collision>
-			<origin xyz="0 0 0.0565" rpy="0 0 0"/>
+			<!-- Используем тот же меш для collision -->
+			<origin xyz="0 0 0" rpy="0 0 0"/>
 			<geometry>
-				<box size="${base_size}"/>
+				<mesh filename="package://rob_box_description/meshes/base_link.stl" scale="0.001 0.001 0.001"/>
 			</geometry>
 		</collision>
-		<inertial>
-			<mass value="${base_mass}"/>
-			<origin xyz="0 0 0.0565"/>
-			<inertia ixx="0.1" ixy="0" ixz="0" iyy="0.1" iyz="0" izz="0.1"/>
-		</inertial>
 	</link>
 	<!-- Макросы -->

Commit message: refactor(urdf): update wheel macro and positions based on Fusion 360 export

File: src/rob_box_description/urdf/rob_box.xacro (robot description, xacro)
@@ -39,63 +39,37 @@
 	</link>
 	<!-- Макросы -->
-	<xacro:macro name="wheel" params="name parent_link origin_xyz rotation_z side">
+	<!-- Wheel Macro - обновлено из Fusion 360 Export (прямое подключение к base_link, без rocker) -->
+	<xacro:macro name="wheel" params="name origin_xyz axis_xyz visual_origin_xyz">
 		<link name="${name}">
-			<visual>
-				<origin xyz="${-0.0035*side} 0 0.1451" rpy="1.5708 0 ${rotation_z}"/>
-				<geometry>
-					<mesh filename="package://rob_box_description/meshes/wheel.stl" scale="0.001 0.001 0.001"/>
+			<!-- Инерциальные параметры из Fusion 360 -->
+			<inertial>
+				<mass value="${wheel_mass}"/>
+				<!-- Inertial origin: смещение центра масс колеса -->
+				<origin xyz="0.0375 0 0"/>
+				<inertia ixx="0.129466" iyy="0.073667" izz="0.073667" ixy="0" iyz="0" ixz="0"/>
+			</inertial>
+			<visual>
+				<!-- Visual origin: offset меша относительно линка (из Fusion 360) -->
+				<origin xyz="${visual_origin_xyz}" rpy="0 0 0"/>
+				<geometry>
+					<mesh filename="package://rob_box_description/meshes/${name}.stl" scale="0.001 0.001 0.001"/>
 				</geometry>
 				<material name="black">
-					<color rgba="0 0 0 1"/>
-				</material>
-			</visual>
-			<collision>
-				<origin xyz="0 ${0.05*side} 0" rpy="1.5708 0 0"/>
-				<geometry>
-					<cylinder radius="${wheel_radius}" length="${wheel_length}"/>
-				</geometry>
-			</collision>
-			<inertial>
-				<mass value="${wheel_mass}"/>
-				<origin xyz="0 0 0"/>
-				<inertia ixx="0.01" ixy="0" ixz="0" iyy="0.01" iyz="0" izz="0.01"/>
-			</inertial>
+					<color rgba="0.1 0.1 0.1 1"/>
+				</material>
+			</visual>
+			<collision>
+				<!-- Collision: используем меш как в Fusion 360 -->
+				<origin xyz="${visual_origin_xyz}" rpy="0 0 0"/>
+				<geometry>
+					<mesh filename="package://rob_box_description/meshes/${name}.stl" scale="0.001 0.001 0.001"/>
+				</geometry>
+			</collision>
 		</link>
 		<joint name="${name}_joint" type="continuous">
-			<parent link="${parent_link}"/>
+			<parent link="base_link"/>
 			<child link="${name}"/>
 			<origin xyz="${origin_xyz}" rpy="0 0 0"/>
-			<axis xyz="0 1 0"/>
-		</joint>
-	</xacro:macro>
-	<xacro:macro name="rocker" params="name side side_x">
-		<link name="${name}">
-			<visual>
-				<origin xyz="0 0 -0.11" rpy="0 3.1416 -1.5708"/>
-				<geometry>
-					<mesh filename="package://rob_box_description/meshes/rocker.stl" scale="${side * 0.001} 0.001 0.001"/>
-				</geometry>
-				<material name="silver">
-					<color rgba="0.5 0.5 0.5 1"/>
-				</material>
-			</visual>
-			<collision>
-				<origin xyz="0 0 0" rpy="0 0 0"/>
-				<geometry>
-					<box size="${rocker_length} ${rocker_width} ${rocker_thickness}"/>
-				</geometry>
-			</collision>
-			<inertial>
-				<mass value="${rocker_mass}"/>
-				<origin xyz="0 0 0"/>
-				<inertia ixx="0.02" ixy="0" ixz="0" iyy="0.02" iyz="0" izz="0.02"/>
-			</inertial>
-		</link>
-		<joint name="${name}_joint" type="fixed">
-			<parent link="base_link"/>
-			<child link="${name}"/>
-			<origin xyz="0 ${side * 0.23048 + side_x} 0.09425" rpy="0 0 0"/>
-			<axis xyz="0 1 0"/>
-			<limit effort="10" velocity="1" lower="-0.3" upper="0.3"/>
+			<axis xyz="${axis_xyz}"/>
 		</joint>
 	</xacro:macro>
@@ -277,11 +251,24 @@
 		</joint>
 	</xacro:macro>
-	<!-- Использование макросов -->
-	<xacro:rocker name="left_rocker" side="1" side_x="-0.05"/>
-	<xacro:rocker name="right_rocker" side="-1" side_x="0.05"/>
-	<xacro:wheel name="left_front_wheel" parent_link="left_rocker" origin_xyz="0.14467 0 -0.11" rotation_z="1.5708" side="1"/>
-	<xacro:wheel name="left_rear_wheel" parent_link="left_rocker" origin_xyz="-0.14467 0 -0.11" rotation_z="1.5708" side="1"/>
-	<xacro:wheel name="right_front_wheel" parent_link="right_rocker" origin_xyz="0.14467 0 -0.11" rotation_z="-1.5708" side="-1"/>
-	<xacro:wheel name="right_rear_wheel" parent_link="right_rocker" origin_xyz="-0.14467 0 -0.11" rotation_z="-1.5708" side="-1"/>
+	<!-- Использование макросов - позиции из Fusion 360 Export -->
+	<!-- Колёса подключены напрямую к base_link (упрощённая модель без rocker-bogie) -->
+	<!-- Left wheels -->
+	<xacro:wheel name="wheel_rear_left_1"
+	             origin_xyz="0.195 0.143797 0.028767"
+	             axis_xyz="1.0 0.0 0.0"
+	             visual_origin_xyz="-0.195 -0.143797 -0.028767"/>
+	<xacro:wheel name="wheel_front_left_1"
+	             origin_xyz="0.195 -0.145731 0.0289"
+	             axis_xyz="1.0 0.0 0.0"
+	             visual_origin_xyz="-0.195 0.145731 -0.0289"/>
+	<!-- Right wheels -->
+	<xacro:wheel name="wheel_front_right_1"
+	             origin_xyz="-0.195967 -0.144669 0.0289"
+	             axis_xyz="-1.0 0.0 0.0"
+	             visual_origin_xyz="0.195967 0.144669 -0.0289"/>
+	<xacro:wheel name="wheel_rear_right_1"
+	             origin_xyz="-0.195 0.143797 0.028767"
+	             axis_xyz="-1.0 0.0 0.0"
+	             visual_origin_xyz="0.195 -0.143797 -0.028767"/>
 	<!-- Сенсоры - позиции из Fusion 360 Export (URDF_ROBBOX.xacro) -->
 	<!-- LiDAR: Rigid 2 joint xyz="-0.000331 0.170806 0.4765" -->
