Commit message: fix: исправлена ориентация робота и имена джойнтов колёс
Co-authored-by: GOODWORKRINKZ <237234482+GOODWORKRINKZ@users.noreply.github.com>

File: src/rob_box_description/urdf/rob_box.xacro (robot description, xacro)
@@ -11,5 +11,16 @@
 	<xacro:property name="rocker_mass" value="3"/>
 	<xacro:property name="base_mass" value="62.64527022934752"/>  <!-- От Fusion 360: 62.65 кг -->
+	<!-- base_footprint - корневой фрейм робота на уровне пола -->
+	<!-- Используется как reference frame в соответствии с REP-120 -->
+	<link name="base_footprint">
+		<visual>
+			<origin xyz="0 0 0" rpy="0 0 0"/>
+			<geometry>
+				<sphere radius="0.001"/>
+			</geometry>
+		</visual>
+	</link>
 	<!-- Основное шасси - обновлено из Fusion 360 Export -->
+	<!-- Повёрнуто на -90° вокруг Z для соответствия ROS convention (X - вперёд, Y - влево) -->
 	<link name="base_link">
 		<!-- Меш base_link.stl из Fusion 360 - нормализован относительно base_link (0,0,0) -->
@@ -38,4 +49,12 @@
 		</collision>
 	</link>
+	<!-- Джойнт base_footprint -> base_link с поворотом на -90° вокруг Z -->
+	<!-- Это исправляет ориентацию: Fusion 360 использует Y вперёд, ROS использует X вперёд -->
+	<joint name="base_footprint_joint" type="fixed">
+		<parent link="base_footprint"/>
+		<child link="base_link"/>
+		<!-- Поворот на -π/2 вокруг Z + поднятие на высоту wheel_radius для base_footprint на уровне пола -->
+		<origin xyz="0 0 ${wheel_radius}" rpy="0 0 -1.5708"/>
+	</joint>
 	<!-- Макросы -->
 	<!-- Wheel Macro - обновлено из Fusion 360 Export (прямое подключение к base_link, без rocker) -->
@@ -253,19 +272,20 @@
 	<!-- Использование макросов - позиции из Fusion 360 Export -->
 	<!-- Колёса подключены напрямую к base_link (упрощённая модель без rocker-bogie) -->
+	<!-- Naming convention: matches robot_controller.yaml (front/rear_left/right_wheel) -->
 	<!-- Left wheels -->
-	<xacro:wheel name="wheel_rear_left_1"
+	<xacro:wheel name="rear_left_wheel"
 	             origin_xyz="0.195 0.143797 0.028767"
 	             axis_xyz="1.0 0.0 0.0"
 	             visual_origin_xyz="-0.195 -0.143797 -0.028767"/>
-	<xacro:wheel name="wheel_front_left_1"
+	<xacro:wheel name="front_left_wheel"
 	             origin_xyz="0.195 -0.145731 0.0289"
 	             axis_xyz="1.0 0.0 0.0"
 	             visual_origin_xyz="-0.195 0.145731 -0.0289"/>
 	<!-- Right wheels -->
-	<xacro:wheel name="wheel_front_right_1"
+	<xacro:wheel name="front_right_wheel"
 	             origin_xyz="-0.195967 -0.144669 0.0289"
 	             axis_xyz="-1.0 0.0 0.0"
 	             visual_origin_xyz="0.195967 0.144669 -0.0289"/>
-	<xacro:wheel name="wheel_rear_right_1"
+	<xacro:wheel name="rear_right_wheel"
 	             origin_xyz="-0.195 0.143797 0.028767"
 	             axis_xyz="-1.0 0.0 0.0"

File: src/rob_box_description/urdf/rob_box_ros2_control.xacro (robot description, xacro)
@@ -19,7 +19,7 @@
     </hardware>
     <!-- ═══════════════════════════════════════════════════════════════ -->
-    <!-- Left Front Wheel -->
+    <!-- Front Left Wheel -->
     <!-- ═══════════════════════════════════════════════════════════════ -->
-    <joint name="left_front_wheel_joint">
+    <joint name="front_left_wheel_joint">
       <command_interface name="velocity">
         <param name="min">-10</param>  <!-- м/с -->
@@ -35,7 +35,7 @@
     </joint>
     <!-- ═══════════════════════════════════════════════════════════════ -->
-    <!-- Right Front Wheel -->
+    <!-- Front Right Wheel -->
     <!-- ═══════════════════════════════════════════════════════════════ -->
-    <joint name="right_front_wheel_joint">
+    <joint name="front_right_wheel_joint">
       <command_interface name="velocity">
         <param name="min">-10</param>
@@ -50,7 +50,7 @@
     </joint>
     <!-- ═══════════════════════════════════════════════════════════════ -->
-    <!-- Left Rear Wheel -->
+    <!-- Rear Left Wheel -->
     <!-- ═══════════════════════════════════════════════════════════════ -->
-    <joint name="left_rear_wheel_joint">
+    <joint name="rear_left_wheel_joint">
       <command_interface name="velocity">
         <param name="min">-10</param>
@@ -65,7 +65,7 @@
     </joint>
     <!-- ═══════════════════════════════════════════════════════════════ -->
-    <!-- Right Rear Wheel -->
+    <!-- Rear Right Wheel -->
     <!-- ═══════════════════════════════════════════════════════════════ -->
-    <joint name="right_rear_wheel_joint">
+    <joint name="rear_right_wheel_joint">
       <command_interface name="velocity">
         <param name="min">-10</param>

Commit message: fix(urdf): correct joint orientation and visual origins in rob_box.xacro

File: src/rob_box_description/urdf/rob_box.xacro (robot description, xacro)
@@ -49,15 +49,16 @@
 		</collision>
 	</link>
-	<!-- Джойнт base_footprint -> base_link с поворотом на -90° вокруг Z -->
-	<!-- Это исправляет ориентацию: Fusion 360 использует Y вперёд, ROS использует X вперёд -->
+	<!-- Джойнт base_footprint -> base_link -->
+	<!-- base_footprint - фрейм на уровне пола, base_link поднят на высоту колеса -->
+	<!-- ВАЖНО: Поворот НЕ применяется - Fusion 360 модель уже в правильной ориентации ROS -->
 	<joint name="base_footprint_joint" type="fixed">
 		<parent link="base_footprint"/>
 		<child link="base_link"/>
-		<!-- Поворот на -π/2 вокруг Z + поднятие на высоту wheel_radius для base_footprint на уровне пола -->
-		<origin xyz="0 0 ${wheel_radius}" rpy="0 0 -1.5708"/>
+		<!-- Только поднятие на высоту wheel_radius для base_footprint на уровне пола -->
+		<origin xyz="0 0 ${wheel_radius}" rpy="0 0 0"/>
 	</joint>
 	<!-- Макросы -->
 	<!-- Wheel Macro - обновлено из Fusion 360 Export (прямое подключение к base_link, без rocker) -->
-	<xacro:macro name="wheel" params="name origin_xyz axis_xyz visual_origin_xyz">
+	<xacro:macro name="wheel" params="name origin_xyz axis_xyz">
 		<link name="${name}">
 			<!-- Инерциальные параметры из Fusion 360 -->
@@ -69,6 +70,6 @@
 			</inertial>
 			<visual>
-				<!-- Visual origin: offset меша относительно линка (из Fusion 360) -->
-				<origin xyz="${visual_origin_xyz}" rpy="0 0 0"/>
+				<!-- Visual origin: меш в локальных координатах линка колеса -->
+				<origin xyz="0 0 0" rpy="0 0 0"/>
 				<geometry>
 					<mesh filename="package://rob_box_description/meshes/${name}.stl" scale="0.001 0.001 0.001"/>
@@ -79,6 +80,6 @@
 			</visual>
 			<collision>
-				<!-- Collision: используем меш как в Fusion 360 -->
-				<origin xyz="${visual_origin_xyz}" rpy="0 0 0"/>
+				<!-- Collision: меш в локальных координатах линка колеса -->
+				<origin xyz="0 0 0" rpy="0 0 0"/>
 				<geometry>
 					<mesh filename="package://rob_box_description/meshes/${name}.stl" scale="0.001 0.001 0.001"/>
@@ -276,19 +277,15 @@
 	<xacro:wheel name="rear_left_wheel"
 	             origin_xyz="0.195 0.143797 0.028767"
-	             axis_xyz="1.0 0.0 0.0"
-	             visual_origin_xyz="-0.195 -0.143797 -0.028767"/>
+	             axis_xyz="1.0 0.0 0.0"/>
 	<xacro:wheel name="front_left_wheel"
 	             origin_xyz="0.195 -0.145731 0.0289"
-	             axis_xyz="1.0 0.0 0.0"
-	             visual_origin_xyz="-0.195 0.145731 -0.0289"/>
+	             axis_xyz="1.0 0.0 0.0"/>
 	<!-- Right wheels -->
 	<xacro:wheel name="front_right_wheel"
 	             origin_xyz="-0.195967 -0.144669 0.0289"
-	             axis_xyz="-1.0 0.0 0.0"
-	             visual_origin_xyz="0.195967 0.144669 -0.0289"/>
+	             axis_xyz="-1.0 0.0 0.0"/>
 	<xacro:wheel name="rear_right_wheel"
 	             origin_xyz="-0.195 0.143797 0.028767"
-	             axis_xyz="-1.0 0.0 0.0"
-	             visual_origin_xyz="0.195 -0.143797 -0.028767"/>
+	             axis_xyz="-1.0 0.0 0.0"/>
 	<!-- Сенсоры - позиции из Fusion 360 Export (URDF_ROBBOX.xacro) -->
 	<!-- LiDAR: Rigid 2 joint xyz="-0.000331 0.170806 0.4765" -->

Commit message: fix(urdf): correct joint orientation and visual origins for wheels in rob_box.xacro

File: src/rob_box_description/urdf/rob_box.xacro (robot description, xacro)
@@ -49,16 +49,15 @@
 		</collision>
 	</link>
-	<!-- Джойнт base_footprint -> base_link -->
-	<!-- base_footprint - фрейм на уровне пола, base_link поднят на высоту колеса -->
-	<!-- ВАЖНО: Поворот НЕ применяется - Fusion 360 модель уже в правильной ориентации ROS -->
+	<!-- Джойнт base_footprint -> base_link с поворотом на -90° вокруг Z -->
+	<!-- Это исправляет ориентацию: Fusion 360 использует Y вперёд, ROS использует X вперёд -->
 	<joint name="base_footprint_joint" type="fixed">
 		<parent link="base_footprint"/>
 		<child link="base_link"/>
-		<!-- Только поднятие на высоту wheel_radius для base_footprint на уровне пола -->
-		<origin xyz="0 0 ${wheel_radius}" rpy="0 0 0"/>
+		<!-- Поворот на -π/2 вокруг Z + поднятие на высоту wheel_radius для base_footprint на уровне пола -->
+		<origin xyz="0 0 ${wheel_radius}" rpy="0 0 -1.5708"/>
 	</joint>
 	<!-- Макросы -->
 	<!-- Wheel Macro - обновлено из Fusion 360 Export (прямое подключение к base_link, без rocker) -->
-	<xacro:macro name="wheel" params="name origin_xyz axis_xyz">
+	<xacro:macro name="wheel" params="name origin_xyz axis_xyz visual_origin_xyz">
 		<link name="${name}">
 			<!-- Инерциальные параметры из Fusion 360 -->
@@ -70,6 +69,6 @@
 			</inertial>
 			<visual>
-				<!-- Visual origin: меш в локальных координатах линка колеса -->
-				<origin xyz="0 0 0" rpy="0 0 0"/>
+				<!-- Visual origin: offset меша относительно линка (из Fusion 360) -->
+				<origin xyz="${visual_origin_xyz}" rpy="0 0 0"/>
 				<geometry>
 					<mesh filename="package://rob_box_description/meshes/${name}.stl" scale="0.001 0.001 0.001"/>
@@ -80,6 +79,6 @@
 			</visual>
 			<collision>
-				<!-- Collision: меш в локальных координатах линка колеса -->
-				<origin xyz="0 0 0" rpy="0 0 0"/>
+				<!-- Collision: используем меш как в Fusion 360 -->
+				<origin xyz="${visual_origin_xyz}" rpy="0 0 0"/>
 				<geometry>
 					<mesh filename="package://rob_box_description/meshes/${name}.stl" scale="0.001 0.001 0.001"/>
@@ -277,15 +276,19 @@
 	<xacro:wheel name="rear_left_wheel"
 	             origin_xyz="0.195 0.143797 0.028767"
-	             axis_xyz="1.0 0.0 0.0"/>
+	             axis_xyz="1.0 0.0 0.0"
+	             visual_origin_xyz="-0.195 -0.143797 -0.028767"/>
 	<xacro:wheel name="front_left_wheel"
 	             origin_xyz="0.195 -0.145731 0.0289"
-	             axis_xyz="1.0 0.0 0.0"/>
+	             axis_xyz="1.0 0.0 0.0"
+	             visual_origin_xyz="-0.195 0.145731 -0.0289"/>
 	<!-- Right wheels -->
 	<xacro:wheel name="front_right_wheel"
 	             origin_xyz="-0.195967 -0.144669 0.0289"
-	             axis_xyz="-1.0 0.0 0.0"/>
+	             axis_xyz="-1.0 0.0 0.0"
+	             visual_origin_xyz="0.195967 0.144669 -0.0289"/>
 	<xacro:wheel name="rear_right_wheel"
 	             origin_xyz="-0.195 0.143797 0.028767"
-	             axis_xyz="-1.0 0.0 0.0"/>
+	             axis_xyz="-1.0 0.0 0.0"
+	             visual_origin_xyz="0.195 -0.143797 -0.028767"/>
 	<!-- Сенсоры - позиции из Fusion 360 Export (URDF_ROBBOX.xacro) -->
 	<!-- LiDAR: Rigid 2 joint xyz="-0.000331 0.170806 0.4765" -->

Commit message: fix(urdf): correct joint orientation for base_footprint_joint in rob_box.xacro

File: src/rob_box_description/urdf/rob_box.xacro (robot description, xacro)
@@ -49,11 +49,11 @@
 		</collision>
 	</link>
-	<!-- Джойнт base_footprint -> base_link с поворотом на -90° вокруг Z -->
+	<!-- Джойнт base_footprint -> base_link с поворотом на +90° вокруг Z -->
 	<!-- Это исправляет ориентацию: Fusion 360 использует Y вперёд, ROS использует X вперёд -->
 	<joint name="base_footprint_joint" type="fixed">
 		<parent link="base_footprint"/>
 		<child link="base_link"/>
-		<!-- Поворот на -π/2 вокруг Z + поднятие на высоту wheel_radius для base_footprint на уровне пола -->
-		<origin xyz="0 0 ${wheel_radius}" rpy="0 0 -1.5708"/>
+		<!-- Поворот на +π/2 вокруг Z + поднятие на высоту wheel_radius для base_footprint на уровне пола -->
+		<origin xyz="0 0 ${wheel_radius}" rpy="0 0 1.5708"/>
 	</joint>
 	<!-- Макросы -->

Commit message: fix(urdf): update imu frame joint orientation in rob_box.xacro

File: src/rob_box_description/urdf/rob_box.xacro (robot description, xacro)
@@ -228,5 +228,5 @@
 			<parent link="${name}"/>
 			<child link="${name}_imu_frame"/>
-			<origin xyz="0 0 0" rpy="0 0 0"/>
+			<origin xyz="0 0 0" rpy="3.14159 0 1.5708"/>
 		</joint>
 	</xacro:macro>

Commit message: fix(urdf): correct joint origin rotation for base_footprint_joint in rob_box.xacro

File: src/rob_box_description/urdf/rob_box.xacro (robot description, xacro)
@@ -55,5 +55,5 @@
 		<child link="base_link"/>
 		<!-- Поворот на +π/2 вокруг Z + поднятие на высоту wheel_radius для base_footprint на уровне пола -->
-		<origin xyz="0 0 ${wheel_radius}" rpy="0 0 1.5708"/>
+		<origin xyz="0 0 ${wheel_radius}" rpy="0 0 0"/>
 	</joint>
 	<!-- Макросы -->

Commit message: fix(urdf): rotate base_link by -90° to align with LiDAR orientation
- LiDAR 0° points forward, but Fusion 360 model is rotated +90°
- Changed base_footprint_joint rotation from 0 to -π/2 (rpy="0 0 -1.5708")
- Now robot model in RViz will match physical orientation
- Based on LaserScan analysis: Rear sector has 244 points (wall behind)

File: src/rob_box_description/urdf/rob_box.xacro (robot description, xacro)
@@ -49,11 +49,11 @@
 		</collision>
 	</link>
-	<!-- Джойнт base_footprint -> base_link с поворотом на +90° вокруг Z -->
-	<!-- Это исправляет ориентацию: Fusion 360 использует Y вперёд, ROS использует X вперёд -->
+	<!-- Джойнт base_footprint -> base_link с поворотом на -90° вокруг Z -->
+	<!-- Исправляет ориентацию: LiDAR 0° = вперёд, но модель в Fusion 360 повёрнута на +90° -->
 	<joint name="base_footprint_joint" type="fixed">
 		<parent link="base_footprint"/>
 		<child link="base_link"/>
-		<!-- Поворот на +π/2 вокруг Z + поднятие на высоту wheel_radius для base_footprint на уровне пола -->
-		<origin xyz="0 0 ${wheel_radius}" rpy="0 0 0"/>
+		<!-- Поворот на -π/2 вокруг Z + поднятие на высоту wheel_radius для base_footprint на уровне пола -->
+		<origin xyz="0 0 ${wheel_radius}" rpy="0 0 -1.5708"/>
 	</joint>
 	<!-- Макросы -->

Commit message: fix(orientation): rotate LiDAR frame instead of base_link
- Reverted base_footprint_joint to rpy="0 0 0" (no rotation)
- Reverted RTAB-Map frame_id back to base_link
- Added origin_rpy="0 0 -1.5708" to LiDAR mount (rotated -90°)
- This aligns LiDAR 0° with robot's forward direction (X axis)
- Robot model orientation now matches odometry arrow in RViz

File: src/rob_box_description/urdf/rob_box.xacro (robot description, xacro)
@@ -49,11 +49,11 @@
 		</collision>
 	</link>
-	<!-- Джойнт base_footprint -> base_link с поворотом на -90° вокруг Z -->
-	<!-- Исправляет ориентацию: LiDAR 0° = вперёд, но модель в Fusion 360 повёрнута на +90° -->
+	<!-- Джойнт base_footprint -> base_link -->
+	<!-- base_footprint на уровне пола, base_link поднят на высоту колеса -->
 	<joint name="base_footprint_joint" type="fixed">
 		<parent link="base_footprint"/>
 		<child link="base_link"/>
-		<!-- Поворот на -π/2 вокруг Z + поднятие на высоту wheel_radius для base_footprint на уровне пола -->
-		<origin xyz="0 0 ${wheel_radius}" rpy="0 0 -1.5708"/>
+		<!-- Поднятие на высоту wheel_radius для base_footprint на уровне пола -->
+		<origin xyz="0 0 ${wheel_radius}" rpy="0 0 0"/>
 	</joint>
 	<!-- Макросы -->
@@ -292,6 +292,6 @@
 	             visual_origin_xyz="0.195 -0.143797 -0.028767"/>
 	<!-- Сенсоры - позиции из Fusion 360 Export (URDF_ROBBOX.xacro) -->
-	<!-- LiDAR: Rigid 2 joint xyz="-0.000331 0.170806 0.4765" -->
-	<xacro:lidar name="lslidar_n10" parent_link="base_link" origin_xyz="-0.000331 0.170806 0.4765" topic_name="/scan"/>
+	<!-- LiDAR: Rigid 2 joint xyz="-0.000331 0.170806 0.4765" (повёрнут на -90° для выравнивания с осью X) -->
+	<xacro:lidar name="lslidar_n10" parent_link="base_link" origin_xyz="-0.000331 0.170806 0.4765" origin_rpy="0 0 -1.5708" topic_name="/scan"/>
 	<!-- OAK-D-Lite камера: Rigid 3 joint xyz="-0.000238 0.115772 0.4595" -->
 	<xacro:oak_d_camera name="camera" parent_link="base_link" origin_xyz="-0.000238 0.115772 0.4595" origin_rpy="0 0 0"/>

Commit message: fix(urdf): add origin_rpy parameter to lidar macro
- Added origin_rpy parameter with default value '0 0 0'
- Updated joint origin to use ${origin_rpy} instead of hardcoded '0 0 0'
- This allows rotating LiDAR frame when instantiating the macro

File: src/rob_box_description/urdf/rob_box.xacro (robot description, xacro)
@@ -94,5 +94,5 @@
 	</xacro:macro>
 	<!-- Сенсоры -->
-	<xacro:macro name="lidar" params="name parent_link origin_xyz topic_name">
+	<xacro:macro name="lidar" params="name parent_link origin_xyz origin_rpy:='0 0 0' topic_name">
 		<link name="${name}">
 			<visual>
@@ -120,5 +120,5 @@
 			<parent link="${parent_link}"/>
 			<child link="${name}"/>
-			<origin xyz="${origin_xyz}" rpy="0 0 0"/>
+			<origin xyz="${origin_xyz}" rpy="${origin_rpy}"/>
 		</joint>
 		<gazebo reference="${name}">

Commit message: fix(urdf): rotate base_link +90° instead of LiDAR
- Reverted LiDAR to origin_rpy="0 0 0" (physically mounted correctly)
- Rotated base_link +90° (rpy="0 0 1.5708") relative to base_footprint
- Fusion 360 model has Y-axis forward, ROS uses X-axis forward
- LiDAR 0° physically points forward along model's Y-axis
- This aligns the visual model with physical robot orientation

File: src/rob_box_description/urdf/rob_box.xacro (robot description, xacro)
@@ -49,11 +49,12 @@
 		</collision>
 	</link>
-	<!-- Джойнт base_footprint -> base_link -->
-	<!-- base_footprint на уровне пола, base_link поднят на высоту колеса -->
+	<!-- Джойнт base_footprint -> base_link с поворотом на +90° вокруг Z -->
+	<!-- Модель из Fusion 360 имеет ось Y вперёд, но ROS использует ось X вперёд -->
+	<!-- LiDAR физически установлен так, что его 0° смотрит вперёд по оси Y модели -->
 	<joint name="base_footprint_joint" type="fixed">
 		<parent link="base_footprint"/>
 		<child link="base_link"/>
-		<!-- Поднятие на высоту wheel_radius для base_footprint на уровне пола -->
-		<origin xyz="0 0 ${wheel_radius}" rpy="0 0 0"/>
+		<!-- Поворот на +π/2 вокруг Z для выравнивания модели с физической ориентацией -->
+		<origin xyz="0 0 ${wheel_radius}" rpy="0 0 1.5708"/>
 	</joint>
 	<!-- Макросы -->
@@ -292,6 +293,6 @@
 	             visual_origin_xyz="0.195 -0.143797 -0.028767"/>
 	<!-- Сенсоры - позиции из Fusion 360 Export (URDF_ROBBOX.xacro) -->
-	<!-- LiDAR: Rigid 2 joint xyz="-0.000331 0.170806 0.4765" (повёрнут на -90° для выравнивания с осью X) -->
-	<xacro:lidar name="lslidar_n10" parent_link="base_link" origin_xyz="-0.000331 0.170806 0.4765" origin_rpy="0 0 -1.5708" topic_name="/scan"/>
+	<!-- LiDAR: Rigid 2 joint xyz="-0.000331 0.170806 0.4765" (без поворота - физически установлен правильно) -->
+	<xacro:lidar name="lslidar_n10" parent_link="base_link" origin_xyz="-0.000331 0.170806 0.4765" topic_name="/scan"/>
 	<!-- OAK-D-Lite камера: Rigid 3 joint xyz="-0.000238 0.115772 0.4595" -->
 	<xacro:oak_d_camera name="camera" parent_link="base_link" origin_xyz="-0.000238 0.115772 0.4595" origin_rpy="0 0 0"/>

Commit message: fix(urdf): rotate base_link by -90° to align robot with physical orientation
- Changed rotation from +90° to -90° (rpy="0 0 -1.5708")
- This rotates the entire robot model (and odometry) by -90°
- Aligns visual model with real-world robot orientation

File: src/rob_box_description/urdf/rob_box.xacro (robot description, xacro)
@@ -49,12 +49,11 @@
 		</collision>
 	</link>
-	<!-- Джойнт base_footprint -> base_link с поворотом на +90° вокруг Z -->
-	<!-- Модель из Fusion 360 имеет ось Y вперёд, но ROS использует ось X вперёд -->
-	<!-- LiDAR физически установлен так, что его 0° смотрит вперёд по оси Y модели -->
+	<!-- Джойнт base_footprint -> base_link с поворотом на -90° вокруг Z -->
+	<!-- Поворот всей модели на -90° для выравнивания с физической ориентацией -->
 	<joint name="base_footprint_joint" type="fixed">
 		<parent link="base_footprint"/>
 		<child link="base_link"/>
-		<!-- Поворот на +π/2 вокруг Z для выравнивания модели с физической ориентацией -->
-		<origin xyz="0 0 ${wheel_radius}" rpy="0 0 1.5708"/>
+		<!-- Поворот на -π/2 (-90°) вокруг Z -->
+		<origin xyz="0 0 ${wheel_radius}" rpy="0 0 -1.5708"/>
 	</joint>
 	<!-- Макросы -->

Commit message: fix(urdf): remove base_link rotation, rotate LiDAR +90°
- Set base_link rotation to 0° (no rotation from base_footprint)
- Rotate LiDAR +90° (rpy="0 0 1.5708") to align with robot forward
- This should align odometry arrow with robot model orientation

File: src/rob_box_description/urdf/rob_box.xacro (robot description, xacro)
@@ -49,11 +49,11 @@
 		</collision>
 	</link>
-	<!-- Джойнт base_footprint -> base_link с поворотом на -90° вокруг Z -->
-	<!-- Поворот всей модели на -90° для выравнивания с физической ориентацией -->
+	<!-- Джойнт base_footprint -> base_link без поворота -->
+	<!-- base_footprint на уровне пола, base_link поднят на высоту колеса -->
 	<joint name="base_footprint_joint" type="fixed">
 		<parent link="base_footprint"/>
 		<child link="base_link"/>
-		<!-- Поворот на -π/2 (-90°) вокруг Z -->
-		<origin xyz="0 0 ${wheel_radius}" rpy="0 0 -1.5708"/>
+		<!-- Без поворота - модель и навигация используют одну ориентацию -->
+		<origin xyz="0 0 ${wheel_radius}" rpy="0 0 0"/>
 	</joint>
 	<!-- Макросы -->
@@ -292,6 +292,6 @@
 	             visual_origin_xyz="0.195 -0.143797 -0.028767"/>
 	<!-- Сенсоры - позиции из Fusion 360 Export (URDF_ROBBOX.xacro) -->
-	<!-- LiDAR: Rigid 2 joint xyz="-0.000331 0.170806 0.4765" (без поворота - физически установлен правильно) -->
-	<xacro:lidar name="lslidar_n10" parent_link="base_link" origin_xyz="-0.000331 0.170806 0.4765" topic_name="/scan"/>
+	<!-- LiDAR: Rigid 2 joint xyz="-0.000331 0.170806 0.4765" (повёрнут на +90° для выравнивания) -->
+	<xacro:lidar name="lslidar_n10" parent_link="base_link" origin_xyz="-0.000331 0.170806 0.4765" origin_rpy="0 0 1.5708" topic_name="/scan"/>
 	<!-- OAK-D-Lite камера: Rigid 3 joint xyz="-0.000238 0.115772 0.4595" -->
 	<xacro:oak_d_camera name="camera" parent_link="base_link" origin_xyz="-0.000238 0.115772 0.4595" origin_rpy="0 0 0"/>
