Commit message: fix(urdf): update LiDAR orientation to align with base_link configuration

File: src/rob_box_description/urdf/rob_box.xacro (robot description, xacro)
@@ -55,5 +55,5 @@
 		<child link="base_link"/>
 		<!-- Без поворота - модель и навигация используют одну ориентацию -->
-		<origin xyz="0 0 ${wheel_radius}" rpy="0 0 0"/>
+		<origin xyz="0 0 ${wheel_radius}" rpy="0 0 1.5708"/>
 	</joint>
 	<!-- Макросы -->
@@ -293,5 +293,5 @@
 	<!-- Сенсоры - позиции из Fusion 360 Export (URDF_ROBBOX.xacro) -->
 	<!-- LiDAR: Rigid 2 joint xyz="-0.000331 0.170806 0.4765" (повёрнут на +90° для выравнивания) -->
-	<xacro:lidar name="lslidar_n10" parent_link="base_link" origin_xyz="-0.000331 0.170806 0.4765" origin_rpy="0 0 1.5708" topic_name="/scan"/>
+	<xacro:lidar name="lslidar_n10" parent_link="base_link" origin_xyz="-0.000331 0.170806 0.4765" origin_rpy="0 0 0" topic_name="/scan"/>
 	<!-- OAK-D-Lite камера: Rigid 3 joint xyz="-0.000238 0.115772 0.4595" -->
 	<xacro:oak_d_camera name="camera" parent_link="base_link" origin_xyz="-0.000238 0.115772 0.4595" origin_rpy="0 0 0"/>

Commit message: fix(urdf): update base_link joint origin to remove rotation for consistent model orientation

File: src/rob_box_description/urdf/rob_box.xacro (robot description, xacro)
@@ -55,5 +55,5 @@
 		<child link="base_link"/>
 		<!-- Без поворота - модель и навигация используют одну ориентацию -->
-		<origin xyz="0 0 ${wheel_radius}" rpy="0 0 1.5708"/>
+		<origin xyz="0 0 ${wheel_radius}" rpy="0 0 0"/>
 	</joint>
 	<!-- Макросы -->

Commit message: fix(urdf): Add -90° Z rotation to base_footprint→base_link
- Lidar data shows correct orientation (front=far wall, rear=furniture)
- But robot model in RViz/RTAB-Map is rotated 90° wrong
- Fusion 360 exported model without ROS convention alignment
- Add rpy="0 0 -1.5708" (-90° around Z) to match real robot orientation

File: src/rob_box_description/urdf/rob_box.xacro (robot description, xacro)
@@ -49,11 +49,12 @@
 		</collision>
 	</link>
-	<!-- Джойнт base_footprint -> base_link без поворота -->
+	<!-- Джойнт base_footprint -> base_link С ПОВОРОТОМ -90° вокруг Z -->
 	<!-- base_footprint на уровне пола, base_link поднят на высоту колеса -->
 	<joint name="base_footprint_joint" type="fixed">
 		<parent link="base_footprint"/>
 		<child link="base_link"/>
-		<!-- Без поворота - модель и навигация используют одну ориентацию -->
-		<origin xyz="0 0 ${wheel_radius}" rpy="0 0 0"/>
+		<!-- Поворот -90° вокруг Z для соответствия ROS convention (X - вперёд, Y - влево) -->
+		<!-- Fusion 360 экспортировал модель с другой ориентацией -->
+		<origin xyz="0 0 ${wheel_radius}" rpy="0 0 -1.5708"/>
 	</joint>
 	<!-- Макросы -->

Commit message: fix(urdf): Rotate base_link visual mesh +90° around Z
- Robot physically faces far wall (front), furniture behind (rear)
- Visual mesh was rotated 90° right (CW) in RViz
- Odometry was rotated 90° left (CCW)
- Apply rpy="0 0 1.5708" (+90° Z) to visual and collision meshes
- Keep base_footprint→base_link joint without rotation for correct TF tree

File: src/rob_box_description/urdf/rob_box.xacro (robot description, xacro)
@@ -32,6 +32,7 @@
 		</inertial>
 		<visual>
-			<!-- Меш без offset - base_link в (0,0,0) как требуется -->
-			<origin xyz="0 0 0" rpy="0 0 0"/>
+			<!-- Меш повернут на +90° вокруг Z для соответствия физической ориентации -->
+			<!-- Fusion 360 экспортировал модель с другой ориентацией относительно ROS convention -->
+			<origin xyz="0 0 0" rpy="0 0 1.5708"/>
 			<geometry>
 				<mesh filename="package://rob_box_description/meshes/base_link.stl" scale="0.001 0.001 0.001"/>
@@ -42,6 +43,6 @@
 		</visual>
 		<collision>
-			<!-- Используем тот же меш для collision -->
-			<origin xyz="0 0 0" rpy="0 0 0"/>
+			<!-- Collision также поворачиваем для соответствия визуализации -->
+			<origin xyz="0 0 0" rpy="0 0 1.5708"/>
 			<geometry>
 				<mesh filename="package://rob_box_description/meshes/base_link.stl" scale="0.001 0.001 0.001"/>
@@ -49,12 +50,11 @@
 		</collision>
 	</link>
-	<!-- Джойнт base_footprint -> base_link С ПОВОРОТОМ -90° вокруг Z -->
+	<!-- Джойнт base_footprint -> base_link БЕЗ ПОВОРОТА -->
 	<!-- base_footprint на уровне пола, base_link поднят на высоту колеса -->
 	<joint name="base_footprint_joint" type="fixed">
 		<parent link="base_footprint"/>
 		<child link="base_link"/>
-		<!-- Поворот -90° вокруг Z для соответствия ROS convention (X - вперёд, Y - влево) -->
-		<!-- Fusion 360 экспортировал модель с другой ориентацией -->
-		<origin xyz="0 0 ${wheel_radius}" rpy="0 0 -1.5708"/>
+		<!-- БЕЗ ПОВОРОТА - одометрия и TF tree должны быть без дополнительных трансформаций -->
+		<origin xyz="0 0 ${wheel_radius}" rpy="0 0 0"/>
 	</joint>
 	<!-- Макросы -->

Commit message: fix(urdf): Add +90° Z rotation to wheel visual/collision meshes
- Wheels meshes from Fusion 360 exported with different orientation
- Add rpy="0 0 1.5708" to wheel macro visual and collision
- Keeps base_link visual rotation, now wheels match
- Lidar and cameras use primitives (cylinder/box), no rotation needed

File: src/rob_box_description/urdf/rob_box.xacro (robot description, xacro)
@@ -1,5 +1,18 @@
 <?xml version="1.0"?>
-<robot name="rob_box" xmlns:xacro="http://www.ros.org/wiki/xacro">
-	<!-- Переменные - обновлено из Fusion 360 Export -->
+<robot name="rob_box" xmlns:xacro="http://www.ros.or		<visual>
+			<!-- Visual origin: offset меша + поворот для соответствия ROS convention -->
+			<origin xyz="${visual_origin_xyz}" rpy="0 0 1.5708"/>
+			<geometry>
+				<mesh filename="package://rob_box_description/meshes/${name}.stl" scale="0.001 0.001 0.001"/>
+			</geometry>
+			<material name="black">
+				<color rgba="0.1 0.1 0.1 1"/>
+			</material>
+		</visual>
+		<collision>
+			<!-- Collision: используем меш как в Fusion 360 + поворот -->
+			<origin xyz="${visual_origin_xyz}" rpy="0 0 1.5708"/>
+			<geometry>
+				<mesh filename="package://rob_box_description/meshes/${name}.stl" scale="0.001 0.001 0.001"/>	<!-- Переменные - обновлено из Fusion 360 Export -->
 	<xacro:property name="base_size" value="0.4757 0.238 0.1885"/>  <!-- Legacy collision box, use mesh instead -->
 	<xacro:property name="wheel_radius" value="0.115"/>

Commit message: fix(urdf): Update visual origin in rob_box.xacro to match ROS convention

File: src/rob_box_description/urdf/rob_box.xacro (robot description, xacro)
@@ -1,4 +1,6 @@
 <?xml version="1.0"?>
-<robot name="rob_box" xmlns:xacro="http://www.ros.or		<visual>
+<robot name="rob_box" xmlns:xacro="http://www.ros.org/wiki/xacro">
+	<!-- Переменные - обновлено из Fusion 360 Export -->
+		<visual>
 			<!-- Visual origin: offset меша + поворот для соответствия ROS convention -->
 			<origin xyz="${visual_origin_xyz}" rpy="0 0 1.5708"/>

Commit message: fix(urdf): Remove visual and collision definitions for base_link to streamline URDF

File: src/rob_box_description/urdf/rob_box.xacro (robot description, xacro)
@@ -2,19 +2,4 @@
 <robot name="rob_box" xmlns:xacro="http://www.ros.org/wiki/xacro">
 	<!-- Переменные - обновлено из Fusion 360 Export -->
-		<visual>
-			<!-- Visual origin: offset меша + поворот для соответствия ROS convention -->
-			<origin xyz="${visual_origin_xyz}" rpy="0 0 1.5708"/>
-			<geometry>
-				<mesh filename="package://rob_box_description/meshes/${name}.stl" scale="0.001 0.001 0.001"/>
-			</geometry>
-			<material name="black">
-				<color rgba="0.1 0.1 0.1 1"/>
-			</material>
-		</visual>
-		<collision>
-			<!-- Collision: используем меш как в Fusion 360 + поворот -->
-			<origin xyz="${visual_origin_xyz}" rpy="0 0 1.5708"/>
-			<geometry>
-				<mesh filename="package://rob_box_description/meshes/${name}.stl" scale="0.001 0.001 0.001"/>	<!-- Переменные - обновлено из Fusion 360 Export -->
 	<xacro:property name="base_size" value="0.4757 0.238 0.1885"/>  <!-- Legacy collision box, use mesh instead -->
 	<xacro:property name="wheel_radius" value="0.115"/>

Commit message: fix(urdf): Add +90° Z rotation to wheel and OAK-D meshes to match base_link orientation

File: src/rob_box_description/urdf/rob_box.xacro (robot description, xacro)
@@ -70,6 +70,6 @@
 			</inertial>
 			<visual>
-				<!-- Visual origin: offset меша относительно линка (из Fusion 360) -->
-				<origin xyz="${visual_origin_xyz}" rpy="0 0 0"/>
+				<!-- Visual origin: offset меша относительно линка + поворот на +90° вокруг Z для соответствия base_link -->
+				<origin xyz="${visual_origin_xyz}" rpy="0 0 1.5708"/>
 				<geometry>
 					<mesh filename="package://rob_box_description/meshes/${name}.stl" scale="0.001 0.001 0.001"/>
@@ -80,6 +80,6 @@
 			</visual>
 			<collision>
-				<!-- Collision: используем меш как в Fusion 360 -->
-				<origin xyz="${visual_origin_xyz}" rpy="0 0 0"/>
+				<!-- Collision: также поворачиваем для соответствия визуализации -->
+				<origin xyz="${visual_origin_xyz}" rpy="0 0 1.5708"/>
 				<geometry>
 					<mesh filename="package://rob_box_description/meshes/${name}.stl" scale="0.001 0.001 0.001"/>
@@ -162,5 +162,6 @@
 		<link name="${name}_link">
 			<visual>
-				<origin xyz="0 0 0" rpy="0 0 0"/>
+				<!-- Поворот на +90° вокруг Z для соответствия base_link ориентации -->
+				<origin xyz="0 0 0" rpy="0 0 1.5708"/>
 				<geometry>
 					<box size="0.097 0.0275 0.0214"/>  <!-- Размеры OAK-D-Lite -->
@@ -171,5 +172,6 @@
 			</visual>
 			<collision>
-				<origin xyz="0 0 0" rpy="0 0 0"/>
+				<!-- Collision также повернут -->
+				<origin xyz="0 0 0" rpy="0 0 1.5708"/>
 				<geometry>
 					<box size="0.097 0.0275 0.0214"/>

Commit message: fix(urdf): Исправление джойнтов колес - вернуть поворот base_link frame
Co-authored-by: GOODWORKRINKZ <237234482+GOODWORKRINKZ@users.noreply.github.com>

File: src/rob_box_description/urdf/rob_box.xacro (robot description, xacro)
@@ -22,5 +22,5 @@
 	</link>
 	<!-- Основное шасси - обновлено из Fusion 360 Export -->
-	<!-- Повёрнуто на -90° вокруг Z для соответствия ROS convention (X - вперёд, Y - влево) -->
+	<!-- Frame base_link повернут на -90° вокруг Z через base_footprint_joint -->
 	<link name="base_link">
 		<!-- Меш base_link.stl из Fusion 360 - нормализован относительно base_link (0,0,0) -->
@@ -32,7 +32,6 @@
 		</inertial>
 		<visual>
-			<!-- Меш повернут на +90° вокруг Z для соответствия физической ориентации -->
-			<!-- Fusion 360 экспортировал модель с другой ориентацией относительно ROS convention -->
-			<origin xyz="0 0 0" rpy="0 0 1.5708"/>
+			<!-- Меш БЕЗ ПОВОРОТА - frame base_link уже повернут через base_footprint_joint -->
+			<origin xyz="0 0 0" rpy="0 0 0"/>
 			<geometry>
 				<mesh filename="package://rob_box_description/meshes/base_link.stl" scale="0.001 0.001 0.001"/>
@@ -43,6 +42,6 @@
 		</visual>
 		<collision>
-			<!-- Collision также поворачиваем для соответствия визуализации -->
-			<origin xyz="0 0 0" rpy="0 0 1.5708"/>
+			<!-- Collision также БЕЗ ПОВОРОТА -->
+			<origin xyz="0 0 0" rpy="0 0 0"/>
 			<geometry>
 				<mesh filename="package://rob_box_description/meshes/base_link.stl" scale="0.001 0.001 0.001"/>
@@ -50,11 +49,12 @@
 		</collision>
 	</link>
-	<!-- Джойнт base_footprint -> base_link БЕЗ ПОВОРОТА -->
+	<!-- Джойнт base_footprint -> base_link С ПОВОРОТОМ -->
 	<!-- base_footprint на уровне пола, base_link поднят на высоту колеса -->
 	<joint name="base_footprint_joint" type="fixed">
 		<parent link="base_footprint"/>
 		<child link="base_link"/>
-		<!-- БЕЗ ПОВОРОТА - одометрия и TF tree должны быть без дополнительных трансформаций -->
-		<origin xyz="0 0 ${wheel_radius}" rpy="0 0 0"/>
+		<!-- ПОВОРОТ НА -90° вокруг Z для соответствия ROS convention (X вперёд) -->
+		<!-- Fusion 360: Y вперёд → ROS: X вперёд → поворот на -90° -->
+		<origin xyz="0 0 ${wheel_radius}" rpy="0 0 -1.5708"/>
 	</joint>
 	<!-- Макросы -->
@@ -70,6 +70,7 @@
 			</inertial>
 			<visual>
-				<!-- Visual origin: offset меша относительно линка + поворот на +90° вокруг Z для соответствия base_link -->
-				<origin xyz="${visual_origin_xyz}" rpy="0 0 1.5708"/>
+				<!-- Visual origin: offset меша относительно линка БЕЗ ПОВОРОТА -->
+				<!-- Frame base_link уже повернут через base_footprint_joint -->
+				<origin xyz="${visual_origin_xyz}" rpy="0 0 0"/>
 				<geometry>
 					<mesh filename="package://rob_box_description/meshes/${name}.stl" scale="0.001 0.001 0.001"/>
@@ -80,6 +81,6 @@
 			</visual>
 			<collision>
-				<!-- Collision: также поворачиваем для соответствия визуализации -->
-				<origin xyz="${visual_origin_xyz}" rpy="0 0 1.5708"/>
+				<!-- Collision также БЕЗ ПОВОРОТА -->
+				<origin xyz="${visual_origin_xyz}" rpy="0 0 0"/>
 				<geometry>
 					<mesh filename="package://rob_box_description/meshes/${name}.stl" scale="0.001 0.001 0.001"/>
@@ -162,6 +163,6 @@
 		<link name="${name}_link">
 			<visual>
-				<!-- Поворот на +90° вокруг Z для соответствия base_link ориентации -->
-				<origin xyz="0 0 0" rpy="0 0 1.5708"/>
+				<!-- БЕЗ ПОВОРОТА - frame base_link уже повернут через base_footprint_joint -->
+				<origin xyz="0 0 0" rpy="0 0 0"/>
 				<geometry>
 					<box size="0.097 0.0275 0.0214"/>  <!-- Размеры OAK-D-Lite -->
@@ -172,6 +173,6 @@
 			</visual>
 			<collision>
-				<!-- Collision также повернут -->
-				<origin xyz="0 0 0" rpy="0 0 1.5708"/>
+				<!-- Collision также БЕЗ ПОВОРОТА -->
+				<origin xyz="0 0 0" rpy="0 0 0"/>
 				<geometry>
 					<box size="0.097 0.0275 0.0214"/>
@@ -273,37 +274,37 @@
 		</joint>
 	</xacro:macro>
-	<!-- Использование макросов - позиции ПЕРЕСЧИТАНЫ для поворота base_link на +90° вокруг Z -->
-	<!-- Формула: new_x = -old_y, new_y = old_x, new_z = old_z -->
+	<!-- Использование макросов - ОРИГИНАЛЬНЫЕ позиции из Fusion 360 -->
+	<!-- Frame base_link повернут на -90° через base_footprint_joint, поэтому позиции остаются как в Fusion -->
 	<!-- Naming convention: matches controller_manager.yaml (left/right_front/rear_wheel) -->
 	<!-- Left wheels -->
-	<!-- Left Rear: Original origin="0.195 0.143797 0.028767" visual="-0.195 -0.143797 -0.028767" -->
+	<!-- Left Rear: Fusion 360 origin="0.195 0.143797 0.028767" visual="-0.195 -0.143797 -0.028767" -->
 	<xacro:wheel name="left_rear_wheel"
-	             origin_xyz="-0.143797 0.195 0.028767"
+	             origin_xyz="0.195 0.143797 0.028767"
 	             axis_xyz="1.0 0.0 0.0"
-	             visual_origin_xyz="0.143797 -0.195 -0.028767"/>
-	<!-- Left Front: Original origin="0.195 -0.145731 0.0289" visual="-0.195 0.145731 -0.0289" -->
+	             visual_origin_xyz="-0.195 -0.143797 -0.028767"/>
+	<!-- Left Front: Fusion 360 origin="0.195 -0.145731 0.0289" visual="-0.195 0.145731 -0.0289" -->
 	<xacro:wheel name="left_front_wheel"
-	             origin_xyz="0.145731 0.195 0.0289"
+	             origin_xyz="0.195 -0.145731 0.0289"
 	             axis_xyz="1.0 0.0 0.0"
-	             visual_origin_xyz="-0.145731 -0.195 -0.0289"/>
+	             visual_origin_xyz="-0.195 0.145731 -0.0289"/>
 	<!-- Right wheels -->
-	<!-- Right Front: Original origin="-0.195967 -0.144669 0.0289" visual="0.195967 0.144669 -0.0289" -->
+	<!-- Right Front: Fusion 360 origin="-0.195967 -0.144669 0.0289" visual="0.195967 0.144669 -0.0289" -->
 	<xacro:wheel name="right_front_wheel"
-	             origin_xyz="0.144669 -0.195967 0.0289"
+	             origin_xyz="-0.195967 -0.144669 0.0289"
 	             axis_xyz="-1.0 0.0 0.0"
-	             visual_origin_xyz="-0.144669 0.195967 -0.0289"/>
-	<!-- Right Rear: Original origin="-0.195 0.143797 0.028767" visual="0.195 -0.143797 -0.028767" -->
+	             visual_origin_xyz="0.195967 0.144669 -0.0289"/>
+	<!-- Right Rear: Fusion 360 origin="-0.195 0.143797 0.028767" visual="0.195 -0.143797 -0.028767" -->
 	<xacro:wheel name="right_rear_wheel"
-	             origin_xyz="-0.143797 -0.195 0.028767"
+	             origin_xyz="-0.195 0.143797 0.028767"
 	             axis_xyz="-1.0 0.0 0.0"
-	             visual_origin_xyz="0.143797 0.195 -0.028767"/>
-	<!-- Сенсоры - позиции ПЕРЕСЧИТАНЫ для поворота base_link на +90° вокруг Z -->
-	<!-- Формула: new_x = -old_y, new_y = old_x, new_z = old_z -->
-	<!-- LiDAR: Original xyz="-0.000331 0.170806 0.4765" → Rotated -->
-	<xacro:lidar name="lslidar_n10" parent_link="base_link" origin_xyz="-0.170806 -0.000331 0.4765" origin_rpy="0 0 0" topic_name="/scan"/>
-	<!-- OAK-D-Lite камера: Original xyz="-0.000238 0.115772 0.4595" → Rotated -->
-	<xacro:oak_d_camera name="camera" parent_link="base_link" origin_xyz="-0.115772 -0.000238 0.4595" origin_rpy="0 0 0"/>
-	<!-- Потолочная USB камера: Original xyz="0.065 0.170663 0.4615" → Rotated -->
-	<xacro:usb_camera name="ceiling_camera" parent_link="base_link" origin_xyz="-0.170663 0.065 0.4615" origin_rpy="0 0 0"/>
+	             visual_origin_xyz="0.195 -0.143797 -0.028767"/>
+	<!-- Сенсоры - ОРИГИНАЛЬНЫЕ позиции из Fusion 360 Export -->
+	<!-- Frame base_link повернут на -90° через base_footprint_joint, поэтому позиции остаются как в Fusion -->
+	<!-- LiDAR: Fusion 360 Rigid 2 joint xyz="-0.000331 0.170806 0.4765" -->
+	<xacro:lidar name="lslidar_n10" parent_link="base_link" origin_xyz="-0.000331 0.170806 0.4765" origin_rpy="0 0 0" topic_name="/scan"/>
+	<!-- OAK-D-Lite камера: Fusion 360 Rigid 3 joint xyz="-0.000238 0.115772 0.4595" -->
+	<xacro:oak_d_camera name="camera" parent_link="base_link" origin_xyz="-0.000238 0.115772 0.4595" origin_rpy="0 0 0"/>
+	<!-- Потолочная USB камера: Fusion 360 xyz="0.065 0.170663 0.4615" -->
+	<xacro:usb_camera name="ceiling_camera" parent_link="base_link" origin_xyz="0.065 0.170663 0.4615" origin_rpy="0 0 0"/>
 	<!-- ros2_control Hardware Interface - VESC Nexus -->
 	<xacro:include filename="rob_box_ros2_control.xacro"/>

Commit message: fix(urdf): rotate wheel axes instead of base_link frame
ПРАВИЛЬНОЕ решение проблемы из комментария @GOODWORKRINKZ:

Проблема: После PR #234 визуал и одометрия не соответствуют физическому роботу
(поворот на 90° влево для одометрии, 90° вправо для визуала).

Причина: PR #234 добавил поворот -90° в base_footprint_joint чтобы исправить оси
колес, но это сломало согласованность визуала/одометрии с физическим роботом.

Решение:
1. Убрал поворот из base_footprint_joint (rpy="0 0 0")
2. Повернул оси колес на 90°:
   - Левые: axis_xyz="1.0 0.0 0.0" → "0.0 1.0 0.0"
   - Правые: axis_xyz="-1.0 0.0 0.0" → "0.0 -1.0 0.0"
3. Вернул base_frame_id обратно на base_link в конфигах

Результат:
✅ Визуал соответствует физическому роботу
✅ Одометрия соответствует физическому роботу
✅ Колеса вращаются правильно (оси повернуты)

См. WHEEL_AXES_FIX_2025-11-20.md для деталей.

Co-authored-by: GOODWORKRINKZ <237234482+GOODWORKRINKZ@users.noreply.github.com>

File: src/rob_box_description/urdf/rob_box.xacro (robot description, xacro)
@@ -22,5 +22,5 @@
 	</link>
 	<!-- Основное шасси - обновлено из Fusion 360 Export -->
-	<!-- Frame base_link повернут на -90° вокруг Z через base_footprint_joint -->
+	<!-- base_link БЕЗ ПОВОРОТА - визуал и одометрия соответствуют физическому роботу -->
 	<link name="base_link">
 		<!-- Меш base_link.stl из Fusion 360 - нормализован относительно base_link (0,0,0) -->
@@ -49,12 +49,11 @@
 		</collision>
 	</link>
-	<!-- Джойнт base_footprint -> base_link С ПОВОРОТОМ -->
+	<!-- Джойнт base_footprint -> base_link БЕЗ ПОВОРОТА -->
 	<!-- base_footprint на уровне пола, base_link поднят на высоту колеса -->
 	<joint name="base_footprint_joint" type="fixed">
 		<parent link="base_footprint"/>
 		<child link="base_link"/>
-		<!-- ПОВОРОТ НА -90° вокруг Z для соответствия ROS convention (X вперёд) -->
-		<!-- Fusion 360: Y вперёд → ROS: X вперёд → поворот на -90° -->
-		<origin xyz="0 0 ${wheel_radius}" rpy="0 0 -1.5708"/>
+		<!-- БЕЗ ПОВОРОТА - визуал и одометрия должны соответствовать физическому роботу -->
+		<origin xyz="0 0 ${wheel_radius}" rpy="0 0 0"/>
 	</joint>
 	<!-- Макросы -->
@@ -275,5 +274,5 @@
 	</xacro:macro>
 	<!-- Использование макросов - ОРИГИНАЛЬНЫЕ позиции из Fusion 360 -->
-	<!-- Frame base_link повернут на -90° через base_footprint_joint, поэтому позиции остаются как в Fusion -->
+	<!-- Оси колес повернуты на 90° для соответствия ROS convention -->
 	<!-- Naming convention: matches controller_manager.yaml (left/right_front/rear_wheel) -->
 	<!-- Left wheels -->
@@ -281,10 +280,10 @@
 	<xacro:wheel name="left_rear_wheel"
 	             origin_xyz="0.195 0.143797 0.028767"
-	             axis_xyz="1.0 0.0 0.0"
+	             axis_xyz="0.0 1.0 0.0"
 	             visual_origin_xyz="-0.195 -0.143797 -0.028767"/>
 	<!-- Left Front: Fusion 360 origin="0.195 -0.145731 0.0289" visual="-0.195 0.145731 -0.0289" -->
 	<xacro:wheel name="left_front_wheel"
 	             origin_xyz="0.195 -0.145731 0.0289"
-	             axis_xyz="1.0 0.0 0.0"
+	             axis_xyz="0.0 1.0 0.0"
 	             visual_origin_xyz="-0.195 0.145731 -0.0289"/>
 	<!-- Right wheels -->
@@ -292,13 +291,12 @@
 	<xacro:wheel name="right_front_wheel"
 	             origin_xyz="-0.195967 -0.144669 0.0289"
-	             axis_xyz="-1.0 0.0 0.0"
+	             axis_xyz="0.0 -1.0 0.0"
 	             visual_origin_xyz="0.195967 0.144669 -0.0289"/>
 	<!-- Right Rear: Fusion 360 origin="-0.195 0.143797 0.028767" visual="0.195 -0.143797 -0.028767" -->
 	<xacro:wheel name="right_rear_wheel"
 	             origin_xyz="-0.195 0.143797 0.028767"
-	             axis_xyz="-1.0 0.0 0.0"
+	             axis_xyz="0.0 -1.0 0.0"
 	             visual_origin_xyz="0.195 -0.143797 -0.028767"/>
 	<!-- Сенсоры - ОРИГИНАЛЬНЫЕ позиции из Fusion 360 Export -->
-	<!-- Frame base_link повернут на -90° через base_footprint_joint, поэтому позиции остаются как в Fusion -->
 	<!-- LiDAR: Fusion 360 Rigid 2 joint xyz="-0.000331 0.170806 0.4765" -->
 	<xacro:lidar name="lslidar_n10" parent_link="base_link" origin_xyz="-0.000331 0.170806 0.4765" origin_rpy="0 0 0" topic_name="/scan"/>
