Commit message: feat(urdf): integrate Fusion 360 corrected export (2e0e5f8)
По запросу @GOODWORKRINKZ: смержен коммит 2e0e5f8 с исправленным экспортом из Fusion 360.

Изменения:
1. Обновлены STL меши из URDF_EXPORT (исправленная модель Fusion 360)
2. Обновлены инерциальные параметры base_link:
   - origin: xyz="-0.025488169162561854 -2.4090750285970683e-05 0.14529190576177384"
   - inertia: ixx="1.926172" iyy="2.829827" (изменена ориентация)
3. Обновлены инерциальные параметры колес:
   - origin: xyz="0 0.0375 0" (было xyz="0.0375 0 0")
   - inertia: ixx="0.073667" iyy="0.129466" (изменена ориентация)
4. Обновлены позиции и оси колес из Fusion (теперь в ROS системе координат):
   - Левые колеса: axis="0.0 1.0 0.0" (было "1.0 0.0 0.0")
   - Правые колеса: axis="0.0 -1.0 0.0" (было "-1.0 0.0 0.0")
5. Обновлены позиции сенсоров согласно новому экспорту

Ключевое изменение: Fusion 360 модель исправлена и теперь экспортируется в правильной ROS системе координат (X вперед, Y влево).

Это исправляет проблему у источника - больше не нужны патчи в URDF!

Co-authored-by: GOODWORKRINKZ <237234482+GOODWORKRINKZ@users.noreply.github.com>

File: src/rob_box_description/urdf/rob_box.xacro (robot description, xacro)
@@ -22,12 +22,12 @@
 	</link>
 	<!-- Основное шасси - обновлено из Fusion 360 Export -->
-	<!-- base_link БЕЗ ПОВОРОТА - визуал и одометрия соответствуют физическому роботу -->
+	<!-- base_link в системе ROS (X вперед, Y влево) - исправленный экспорт из Fusion -->
 	<link name="base_link">
 		<!-- Меш base_link.stl из Fusion 360 - нормализован относительно base_link (0,0,0) -->
 		<inertial>
-			<!-- Инерциальные параметры из Fusion 360 -->
-			<origin xyz="-2.4090750286344156e-05 0.025488169162562517 0.14529190576177464" rpy="0 0 0"/>
+			<!-- Инерциальные параметры из Fusion 360 (исправленный экспорт 2e0e5f8) -->
+			<origin xyz="-0.025488169162561854 -2.4090750285970683e-05 0.14529190576177384" rpy="0 0 0"/>
 			<mass value="${base_mass}"/>
-			<inertia ixx="2.829827" iyy="1.926172" izz="3.653023" ixy="-0.001791" iyz="-0.302171" ixz="-0.001655"/>
+			<inertia ixx="1.926172" iyy="2.829827" izz="3.653023" ixy="0.001791" iyz="-0.001655" ixz="0.302171"/>
 		</inertial>
 		<visual>
@@ -58,13 +58,13 @@
 	</joint>
 	<!-- Макросы -->
-	<!-- Wheel Macro - обновлено из Fusion 360 Export (прямое подключение к base_link, без rocker) -->
+	<!-- Wheel Macro - обновлено из Fusion 360 Export (исправленный экспорт 2e0e5f8) -->
 	<xacro:macro name="wheel" params="name origin_xyz axis_xyz visual_origin_xyz">
 		<link name="${name}">
-			<!-- Инерциальные параметры из Fusion 360 -->
+			<!-- Инерциальные параметры из Fusion 360 (исправленный экспорт) -->
 			<inertial>
 				<mass value="${wheel_mass}"/>
 				<!-- Inertial origin: смещение центра масс колеса -->
-				<origin xyz="0.0375 0 0"/>
-				<inertia ixx="0.129466" iyy="0.073667" izz="0.073667" ixy="0" iyz="0" ixz="0"/>
+				<origin xyz="0 0.0375 0"/>
+				<inertia ixx="0.073667" iyy="0.129466" izz="0.073667" ixy="0" iyz="0" ixz="0"/>
 			</inertial>
 			<visual>
@@ -273,36 +273,36 @@
 		</joint>
 	</xacro:macro>
-	<!-- Использование макросов - ОРИГИНАЛЬНЫЕ позиции из Fusion 360 -->
-	<!-- Оси колес в системе Fusion 360 (X-axis) -->
+	<!-- Использование макросов - ОБНОВЛЕНО из Fusion 360 (исправленный экспорт 2e0e5f8) -->
+	<!-- Система координат теперь соответствует ROS: X вперед, Y влево -->
 	<!-- Naming convention: matches controller_manager.yaml (left/right_front/rear_wheel) -->
 	<!-- Left wheels -->
-	<!-- Left Rear: Fusion 360 origin="0.195 0.143797 0.028767" visual="-0.195 -0.143797 -0.028767" -->
+	<!-- Left Rear: Fusion 360 исправленный экспорт origin="-0.143797 0.195 0.028767" -->
 	<xacro:wheel name="left_rear_wheel"
-	             origin_xyz="0.195 0.143797 0.028767"
-	             axis_xyz="1.0 0.0 0.0"
-	             visual_origin_xyz="-0.195 -0.143797 -0.028767"/>
-	<!-- Left Front: Fusion 360 origin="0.195 -0.145731 0.0289" visual="-0.195 0.145731 -0.0289" -->
+	             origin_xyz="-0.143797 0.195 0.028767"
+	             axis_xyz="0.0 1.0 0.0"
+	             visual_origin_xyz="0.143797 -0.195 -0.028767"/>
+	<!-- Left Front: Fusion 360 исправленный экспорт origin="0.145731 0.195 0.0289" -->
 	<xacro:wheel name="left_front_wheel"
-	             origin_xyz="0.195 -0.145731 0.0289"
-	             axis_xyz="1.0 0.0 0.0"
-	             visual_origin_xyz="-0.195 0.145731 -0.0289"/>
+	             origin_xyz="0.145731 0.195 0.0289"
+	             axis_xyz="0.0 1.0 0.0"
+	             visual_origin_xyz="-0.145731 -0.195 -0.0289"/>
 	<!-- Right wheels -->
-	<!-- Right Front: Fusion 360 origin="-0.195967 -0.144669 0.0289" visual="0.195967 0.144669 -0.0289" -->
+	<!-- Right Front: Fusion 360 исправленный экспорт origin="0.144669 -0.195967 0.0289" -->
 	<xacro:wheel name="right_front_wheel"
-	             origin_xyz="-0.195967 -0.144669 0.0289"
-	             axis_xyz="-1.0 0.0 0.0"
-	             visual_origin_xyz="0.195967 0.144669 -0.0289"/>
-	<!-- Right Rear: Fusion 360 origin="-0.195 0.143797 0.028767" visual="0.195 -0.143797 -0.028767" -->
+	             origin_xyz="0.144669 -0.195967 0.0289"
+	             axis_xyz="0.0 -1.0 0.0"
+	             visual_origin_xyz="-0.144669 0.195967 -0.0289"/>
+	<!-- Right Rear: Fusion 360 исправленный экспорт origin="-0.143797 -0.195 0.028767" -->
 	<xacro:wheel name="right_rear_wheel"
-	             origin_xyz="-0.195 0.143797 0.028767"
-	             axis_xyz="-1.0 0.0 0.0"
-	             visual_origin_xyz="0.195 -0.143797 -0.028767"/>
-	<!-- Сенсоры - ОРИГИНАЛЬНЫЕ позиции из Fusion 360 Export -->
-	<!-- LiDAR: Fusion 360 Rigid 2 joint xyz="-0.000331 0.170806 0.4765" -->
-	<xacro:lidar name="lslidar_n10" parent_link="base_link" origin_xyz="-0.000331 0.170806 0.4765" origin_rpy="0 0 0" topic_name="/scan"/>
-	<!-- OAK-D-Lite камера: Fusion 360 Rigid 3 joint xyz="-0.000238 0.115772 0.4595" -->
-	<xacro:oak_d_camera name="camera" parent_link="base_link" origin_xyz="-0.000238 0.115772 0.4595" origin_rpy="0 0 0"/>
-	<!-- Потолочная USB камера: Fusion 360 xyz="0.065 0.170663 0.4615" -->
-	<xacro:usb_camera name="ceiling_camera" parent_link="base_link" origin_xyz="0.065 0.170663 0.4615" origin_rpy="0 0 0"/>
+	             origin_xyz="-0.143797 -0.195 0.028767"
+	             axis_xyz="0.0 -1.0 0.0"
+	             visual_origin_xyz="0.143797 0.195 -0.028767"/>
+	<!-- Сенсоры - ОБНОВЛЕНО из Fusion 360 Export (исправленный экспорт 2e0e5f8) -->
+	<!-- LiDAR: Fusion 360 исправленный экспорт xyz="-0.170806 -0.000331 0.4765" -->
+	<xacro:lidar name="lslidar_n10" parent_link="base_link" origin_xyz="-0.170806 -0.000331 0.4765" origin_rpy="0 0 0" topic_name="/scan"/>
+	<!-- OAK-D-Lite камера: Fusion 360 исправленный экспорт xyz="-0.115772 -0.000238 0.4595" -->
+	<xacro:oak_d_camera name="camera" parent_link="base_link" origin_xyz="-0.115772 -0.000238 0.4595" origin_rpy="0 0 0"/>
+	<!-- Потолочная USB камера: Fusion 360 исправленный экспорт xyz="-0.170663 -0.065 0.4615" -->
+	<xacro:usb_camera name="ceiling_camera" parent_link="base_link" origin_xyz="-0.170663 -0.065 0.4615" origin_rpy="0 0 0"/>
 	<!-- ros2_control Hardware Interface - VESC Nexus -->
 	<xacro:include filename="rob_box_ros2_control.xacro"/>

Commit message: fix(urdf): use camera_rpi.stl mesh in usb_camera macro
По вопросу @GOODWORKRINKZ: camera_rpi.stl не использовался.

Проблема: Макрос usb_camera использовал простой box вместо STL меша camera_rpi.stl

Решение:
- Заменен box на mesh: camera_rpi.stl
- Обновлены инерциальные параметры из экспорта Fusion:
  * mass: 0.029 кг (29g)
  * origin: xyz="0 0 0.008"
  * inertia обновлена

Теперь потолочная RPI камера использует правильный STL меш из Fusion 360.

Co-authored-by: GOODWORKRINKZ <237234482+GOODWORKRINKZ@users.noreply.github.com>

File: src/rob_box_description/urdf/rob_box.xacro (robot description, xacro)
@@ -241,5 +241,5 @@
 				<origin xyz="0 0 0" rpy="0 0 0"/>
 				<geometry>
-					<box size="0.03 0.03 0.02"/>  <!-- Размеры generic USB камеры -->
+					<mesh filename="package://rob_box_description/meshes/camera_rpi.stl" scale="0.001 0.001 0.001"/>
 				</geometry>
 				<material name="black">
@@ -250,11 +250,11 @@
 				<origin xyz="0 0 0" rpy="0 0 0"/>
 				<geometry>
-					<box size="0.03 0.03 0.02"/>
+					<mesh filename="package://rob_box_description/meshes/camera_rpi.stl" scale="0.001 0.001 0.001"/>
 				</geometry>
 			</collision>
 			<inertial>
-				<mass value="0.05"/>  <!-- ~50g -->
-				<origin xyz="0 0 0"/>
-				<inertia ixx="0.00001" ixy="0" ixz="0" iyy="0.00001" iyz="0" izz="0.00001"/>
+				<mass value="0.029"/>  <!-- 29g из экспорта Fusion -->
+				<origin xyz="0 0 0.008"/>  <!-- Из экспорта Fusion -->
+				<inertia ixx="0.000002" ixy="0" ixz="0" iyy="0.000002" iyz="0" izz="0.000001"/>
 			</inertial>
 		</link>

Commit message: fix(urdf): add visual/collision offset for camera_rpi mesh
По feedback @GOODWORKRINKZ: меш RPI камеры "улетел в космос", во Fusion стоит нормально.

Проблема: В экспорте Fusion у camera_rpi_1 есть visual offset для меша:
xyz="0.170663 -0.065 -0.4615", который компенсирует позицию joint-а.
Макрос usb_camera не учитывал этот offset.

Решение:
- Добавлен visual origin: xyz="0.170663 -0.065 -0.4615" (из экспорта Fusion)
- Добавлен collision origin: xyz="0.170663 -0.065 -0.4615"

Теперь меш RPI камеры в правильной позиции относительно линка.

Co-authored-by: GOODWORKRINKZ <237234482+GOODWORKRINKZ@users.noreply.github.com>

File: src/rob_box_description/urdf/rob_box.xacro (robot description, xacro)
@@ -239,5 +239,6 @@
 		<link name="${name}_link">
 			<visual>
-				<origin xyz="0 0 0" rpy="0 0 0"/>
+				<!-- Visual offset из экспорта Fusion (компенсация позиции меша) -->
+				<origin xyz="0.170663 -0.065 -0.4615" rpy="0 0 0"/>
 				<geometry>
 					<mesh filename="package://rob_box_description/meshes/camera_rpi.stl" scale="0.001 0.001 0.001"/>
@@ -248,5 +249,6 @@
 			</visual>
 			<collision>
-				<origin xyz="0 0 0" rpy="0 0 0"/>
+				<!-- Collision offset из экспорта Fusion -->
+				<origin xyz="0.170663 -0.065 -0.4615" rpy="0 0 0"/>
 				<geometry>
 					<mesh filename="package://rob_box_description/meshes/camera_rpi.stl" scale="0.001 0.001 0.001"/>

Commit message: fix(urdf): add 90° rotation around X for camera_rpi mesh
По feedback @GOODWORKRINKZ: меш стал как надо, но повернут на 90° по оси X.

Проблема: Меш camera_rpi.stl в STL файле ориентирован с поворотом на 90° по X
относительно ожидаемой ориентации.

Решение:
- Добавлен поворот rpy="1.5708 0 0" (90° вокруг X) в visual origin
- Добавлен поворот rpy="1.5708 0 0" в collision origin

Теперь меш RPI камеры в правильной позиции и правильной ориентации.

Co-authored-by: GOODWORKRINKZ <237234482+GOODWORKRINKZ@users.noreply.github.com>

File: src/rob_box_description/urdf/rob_box.xacro (robot description, xacro)
@@ -239,6 +239,6 @@
 		<link name="${name}_link">
 			<visual>
-				<!-- Visual offset из экспорта Fusion (компенсация позиции меша) -->
-				<origin xyz="0.170663 -0.065 -0.4615" rpy="0 0 0"/>
+				<!-- Visual offset из экспорта Fusion + поворот на 90° по X (ориентация меша в STL) -->
+				<origin xyz="0.170663 -0.065 -0.4615" rpy="1.5708 0 0"/>
 				<geometry>
 					<mesh filename="package://rob_box_description/meshes/camera_rpi.stl" scale="0.001 0.001 0.001"/>
@@ -249,6 +249,6 @@
 			</visual>
 			<collision>
-				<!-- Collision offset из экспорта Fusion -->
-				<origin xyz="0.170663 -0.065 -0.4615" rpy="0 0 0"/>
+				<!-- Collision offset из экспорта Fusion + поворот на 90° по X -->
+				<origin xyz="0.170663 -0.065 -0.4615" rpy="1.5708 0 0"/>
 				<geometry>
 					<mesh filename="package://rob_box_description/meshes/camera_rpi.stl" scale="0.001 0.001 0.001"/>

Commit message: fix(urdf): align camera origins with Fusion 360 export
По запросу @GOODWORKRINKZ: тщательный ревью камер показал что origin не совпадают с экспортом.

Проблемы:
1. OAK-D использовал box вместо camera_oak.stl
2. OAK-D joint имел rpy="1.5708 0 1.5708" вместо "0 0 0" из экспорта
3. RPI joint имел rpy="0 0 1.5708" вместо "0 0 0" из экспорта
4. RPI visual имел лишний поворот rpy="1.5708 0 0"

Решение - точное соответствие экспорту Fusion:
- OAK-D: меш camera_oak.stl, visual offset xyz="0.115772 0.000238 -0.4595"
- OAK-D: инерция из экспорта (350g)
- OAK-D joint: xyz="-0.115772 -0.000238 0.4595" rpy="0 0 0"
- RPI: visual offset xyz="0.170663 -0.065 -0.4615" rpy="0 0 0"
- RPI joint: xyz="-0.170663 0.065 0.4615" rpy="0 0 0"

Теперь origins полностью совпадают с экспортом Fusion 360.

Co-authored-by: GOODWORKRINKZ <237234482+GOODWORKRINKZ@users.noreply.github.com>

File: src/rob_box_description/urdf/rob_box.xacro (robot description, xacro)
@@ -162,8 +162,8 @@
 		<link name="${name}_link">
 			<visual>
-				<!-- БЕЗ ПОВОРОТА - frame base_link уже повернут через base_footprint_joint -->
-				<origin xyz="0 0 0" rpy="0 0 0"/>
-				<geometry>
-					<box size="0.097 0.0275 0.0214"/>  <!-- Размеры OAK-D-Lite -->
+				<!-- Visual offset из экспорта Fusion (компенсация позиции меша) -->
+				<origin xyz="0.115772 0.000238 -0.4595" rpy="0 0 0"/>
+				<geometry>
+					<mesh filename="package://rob_box_description/meshes/camera_oak.stl" scale="0.001 0.001 0.001"/>
 				</geometry>
 				<material name="dark_grey">
@@ -172,14 +172,14 @@
 			</visual>
 			<collision>
-				<!-- Collision также БЕЗ ПОВОРОТА -->
-				<origin xyz="0 0 0" rpy="0 0 0"/>
-				<geometry>
-					<box size="0.097 0.0275 0.0214"/>
+				<!-- Collision offset из экспорта Fusion -->
+				<origin xyz="0.115772 0.000238 -0.4595" rpy="0 0 0"/>
+				<geometry>
+					<mesh filename="package://rob_box_description/meshes/camera_oak.stl" scale="0.001 0.001 0.001"/>
 				</geometry>
 			</collision>
 			<inertial>
-				<mass value="0.061"/>  <!-- 61g вес OAK-D-Lite -->
-				<origin xyz="0 0 0"/>
-				<inertia ixx="0.00001" ixy="0" ixz="0" iyy="0.00001" iyz="0" izz="0.00001"/>
+				<mass value="0.350"/>  <!-- 350g из экспорта Fusion -->
+				<origin xyz="0.00875 0.015 0"/>  <!-- Из экспорта Fusion -->
+				<inertia ixx="0.000264" ixy="0" ixz="0" iyy="0.000032" iyz="0" izz="0.00025"/>
 			</inertial>
 		</link>
@@ -239,6 +239,6 @@
 		<link name="${name}_link">
 			<visual>
-				<!-- Visual offset из экспорта Fusion + поворот на 90° по X (ориентация меша в STL) -->
-				<origin xyz="0.170663 -0.065 -0.4615" rpy="1.5708 0 0"/>
+				<!-- Visual offset из экспорта Fusion (компенсация позиции меша) -->
+				<origin xyz="0.170663 -0.065 -0.4615" rpy="0 0 0"/>
 				<geometry>
 					<mesh filename="package://rob_box_description/meshes/camera_rpi.stl" scale="0.001 0.001 0.001"/>
@@ -249,6 +249,6 @@
 			</visual>
 			<collision>
-				<!-- Collision offset из экспорта Fusion + поворот на 90° по X -->
-				<origin xyz="0.170663 -0.065 -0.4615" rpy="1.5708 0 0"/>
+				<!-- Collision offset из экспорта Fusion -->
+				<origin xyz="0.170663 -0.065 -0.4615" rpy="0 0 0"/>
 				<geometry>
 					<mesh filename="package://rob_box_description/meshes/camera_rpi.stl" scale="0.001 0.001 0.001"/>
@@ -303,10 +303,8 @@
 	<!-- LiDAR: Fusion 360 исправленный экспорт xyz="-0.170806 -0.000331 0.4765" -->
 	<xacro:lidar name="lslidar_n10" parent_link="base_link" origin_xyz="-0.170806 -0.000331 0.4765" origin_rpy="0 0 0" topic_name="/scan"/>
-	<!-- OAK-D-Lite камера: Fusion 360 исправленный экспорт xyz="-0.115772 -0.000238 0.4595" -->
-	<!-- Поворот на 90° вокруг Z для компенсации изменения системы координат -->
-	<xacro:oak_d_camera name="camera" parent_link="base_link" origin_xyz="-0.115772 -0.000238 0.4595" origin_rpy="1.5708 0 1.5708"/>
-	<!-- Потолочная USB камера: Fusion 360 исправленный экспорт xyz="-0.170663 0.065 0.4615" -->
-	<!-- Потолочная камера смотрит вверх, поворот: -90° вокруг Y (Z вверх) + 90° вокруг Z (компенсация) -->
-	<xacro:usb_camera name="ceiling_camera" parent_link="base_link" origin_xyz="-0.170663 0.065 0.4615" origin_rpy="0 0 1.5708"/>
+	<!-- OAK-D-Lite камера: Fusion 360 исправленный экспорт xyz="-0.115772 -0.000238 0.4595" rpy="0 0 0" -->
+	<xacro:oak_d_camera name="camera" parent_link="base_link" origin_xyz="-0.115772 -0.000238 0.4595" origin_rpy="0 0 0"/>
+	<!-- Потолочная USB камера: Fusion 360 исправленный экспорт xyz="-0.170663 0.065 0.4615" rpy="0 0 0" -->
+	<xacro:usb_camera name="ceiling_camera" parent_link="base_link" origin_xyz="-0.170663 0.065 0.4615" origin_rpy="0 0 0"/>
 	<!-- ros2_control Hardware Interface - VESC Nexus -->
 	<xacro:include filename="rob_box_ros2_control.xacro"/>

Commit message: fix(odometry): calibrate wheel_radius 0.115→0.138 (1.2x factor)
Based on 4.45m measurement test:
- Real distance: 4.45m (tape measure) / 4.37m (lidar)
- Odometry showed: 3.67m
- Calibration factor: 4.45/3.67 = 1.21

Updated wheel_radius from 0.115 to 0.138 (0.115 × 1.2) in:
- docker/main/config/controllers/controller_manager.yaml
- docker/main/config/vesc_nexus/vesc_config.yaml
- docker/main/config/vesc_nexus/robot_controller.yaml
- src/rob_box_description/urdf/rob_box.xacro
- src/rob_box_description/urdf/rob_box_ros2_control.xacro
- src/vesc_nexus (submodule updated)

File: src/rob_box_description/urdf/rob_box.xacro (robot description, xacro)
@@ -3,5 +3,5 @@
 	<!-- Переменные - обновлено из Fusion 360 Export -->
 	<xacro:property name="base_size" value="0.4757 0.238 0.1885"/>  <!-- Legacy collision box, use mesh instead -->
-	<xacro:property name="wheel_radius" value="0.115"/>
+	<xacro:property name="wheel_radius" value="0.138"/>  <!-- Калибровочный: 0.115 × 1.2 -->
 	<xacro:property name="wheel_length" value="0.05"/>
 	<xacro:property name="rocker_length" value="0.28934"/>

File: src/rob_box_description/urdf/rob_box_ros2_control.xacro (robot description, xacro)
@@ -2,5 +2,9 @@
 <!--
   rob_box_ros2_control.xacro
-  ros2_control интеграция с VESC Nexus hardware interface
+  ros2_control интеграция с VESC Nex      <param name="can_id">124</param>
+      <param name="poles">30</param>
+      <param name="min_erpm">24</param>
+      <param name="wheel_radius">0.138</param>
+      <param name="max_rps">11.93</param>          <!-- Калибровка: об/сек при duty=100% -->rdware interface
   Определяет 4 колеса с VESC моторами через CAN
 -->
@@ -16,5 +20,5 @@
       <param name="publish_rate">50.0</param>
       <!-- Default wheel radius (может быть переопределен для каждого колеса) -->
-      <param name="wheel_radius">0.115</param>
+      <param name="wheel_radius">0.138</param>
       <!-- Минимальный duty cycle для преодоления мёртвой зоны VESC -->
       <!-- Калибровка 2025-12-14: duty=0.05 еле крутится, duty=0.10 нормально -->
@@ -36,5 +40,5 @@
       <param name="poles">30</param>               <!-- Количество полюсов мотора -->
       <param name="min_erpm">24</param>           <!-- Минимальный ERPM для движения -->
-      <param name="wheel_radius">0.115</param>     <!-- Радиус колеса (м) -->
+      <param name="wheel_radius">0.138</param>     <!-- Калиброван: 0.115 × 1.2 = 0.138 -->
       <param name="max_rps">11.83</param>          <!-- Калибровка: об/сек при duty=100% -->
     </joint>
@@ -52,5 +56,5 @@
       <param name="poles">30</param>
       <param name="min_erpm">24</param>
-      <param name="wheel_radius">0.115</param>
+      <param name="wheel_radius">0.138</param>
       <param name="max_rps">11.53</param>          <!-- Калибровка: об/сек при duty=100% -->
     </joint>
@@ -68,5 +72,5 @@
       <param name="poles">30</param>
       <param name="min_erpm">24</param>
-      <param name="wheel_radius">0.115</param>
+      <param name="wheel_radius">0.138</param>
       <param name="max_rps">11.70</param>          <!-- Калибровка: об/сек при duty=100% -->
     </joint>
@@ -84,5 +88,5 @@
       <param name="poles">30</param>
       <param name="min_erpm">24</param>
-      <param name="wheel_radius">0.115</param>
+      <param name="wheel_radius">0.138</param>
       <param name="max_rps">11.93</param>          <!-- Калибровка: об/сек при duty=100% -->
     </joint>
