Commit message: calibration(vesc): update wheel params for 9" geared wheels
- wheel_radius: 0.138 → 0.1143 m (9 inch diameter)
- wheel_max_rps: [11.83,11.93,11.70,11.53] → [6.5,6.5,6.5,6.5]
  measured 2026-02-23: FL=7.22, FR=6.64, RL=7.10, RR=7.16
  using 6.5 (below FR minimum, no duty overflow)
- Updated: rob_box.xacro, rob_box_ros2_control.xacro,
  controller_manager.yaml, robot_controller.yaml, vesc_config.yaml

File: src/rob_box_description/urdf/rob_box.xacro (robot description, xacro)
@@ -3,5 +3,5 @@
 	<!-- Переменные - обновлено из Fusion 360 Export -->
 	<xacro:property name="base_size" value="0.4757 0.238 0.1885"/>  <!-- Legacy collision box, use mesh instead -->
-	<xacro:property name="wheel_radius" value="0.138"/>  <!-- Калибровочный: 0.115 × 1.2 -->
+	<xacro:property name="wheel_radius" value="0.1143"/>  <!-- Замер 2026-02-23: 9" колёса с редукторами -->
 	<xacro:property name="wheel_length" value="0.05"/>
 	<xacro:property name="rocker_length" value="0.28934"/>

File: src/rob_box_description/urdf/rob_box_ros2_control.xacro (robot description, xacro)
@@ -15,6 +15,6 @@
       <param name="can_interface">can0</param>
       <param name="publish_rate">50.0</param>
-      <!-- Default wheel radius (может быть переопределен для каждого колеса) -->
-      <param name="wheel_radius">0.138</param>
+      <!-- Default wheel radius: 9" колёса с редукторами, замер 2026-02-23 -->
+      <param name="wheel_radius">0.1143</param>
       <!-- Минимальный duty cycle для преодоления мёртвой зоны VESC -->
       <!-- Калибровка 2025-12-14: duty=0.05 еле крутится, duty=0.10 нормально -->
@@ -43,6 +43,6 @@
       <param name="poles">30</param>               <!-- Количество полюсов мотора -->
       <param name="min_erpm">24</param>           <!-- Минимальный ERPM для движения -->
-      <param name="wheel_radius">0.138</param>     <!-- Калиброван: 0.115 × 1.2 = 0.138 -->
-      <param name="max_rps">11.83</param>          <!-- Калибровка: об/сек при duty=100% -->
+      <param name="wheel_radius">0.1143</param>    <!-- Замер 2026-02-23: 9" с редуктором -->
+      <param name="max_rps">6.5</param>             <!-- Замер 2026-02-23: FL=7.22, используем 6.5 -->
     </joint>
     <!-- ═══════════════════════════════════════════════════════════════ -->
@@ -59,6 +59,6 @@
       <param name="poles">30</param>
       <param name="min_erpm">24</param>
-      <param name="wheel_radius">0.138</param>
-      <param name="max_rps">11.53</param>          <!-- Калибровка: об/сек при duty=100% -->
+      <param name="wheel_radius">0.1143</param>    <!-- Замер 2026-02-23: 9" с редуктором -->
+      <param name="max_rps">6.5</param>             <!-- Замер 2026-02-23: RR=7.16, используем 6.5 -->
     </joint>
     <!-- ═══════════════════════════════════════════════════════════════ -->
@@ -75,6 +75,6 @@
       <param name="poles">30</param>
       <param name="min_erpm">24</param>
-      <param name="wheel_radius">0.138</param>
-      <param name="max_rps">11.70</param>          <!-- Калибровка: об/сек при duty=100% -->
+      <param name="wheel_radius">0.1143</param>    <!-- Замер 2026-02-23: 9" с редуктором -->
+      <param name="max_rps">6.5</param>             <!-- Замер 2026-02-23: RL=7.10, используем 6.5 -->
     </joint>
     <!-- ═══════════════════════════════════════════════════════════════ -->
@@ -91,6 +91,6 @@
       <param name="poles">30</param>
       <param name="min_erpm">24</param>
-      <param name="wheel_radius">0.138</param>
-      <param name="max_rps">11.93</param>          <!-- Калибровка: об/сек при duty=100% -->
+      <param name="wheel_radius">0.1143</param>    <!-- Замер 2026-02-23: 9" с редуктором -->
+      <param name="max_rps">6.5</param>             <!-- Замер 2026-02-23: FR=6.64, используем 6.5 -->
     </joint>
   </ros2_control>

Commit message: feat(camera): add compatibility aliases for depthai_ros_driver color frame naming

File: src/rob_box_description/urdf/rob_box.xacro (robot description, xacro)
@@ -212,4 +212,17 @@
 			<origin xyz="0 0 0" rpy="-1.5708 0 -1.5708"/>
 		</joint>
+		<!-- Compatibility aliases for current depthai_ros_driver color frame naming -->
+		<link name="${name}_color_frame"/>
+		<joint name="${name}_color_frame_joint" type="fixed">
+			<parent link="${name}_rgb_camera_frame"/>
+			<child link="${name}_color_frame"/>
+			<origin xyz="0 0 0" rpy="0 0 0"/>
+		</joint>
+		<link name="${name}_color_optical_frame"/>
+		<joint name="${name}_color_optical_frame_joint" type="fixed">
+			<parent link="${name}_rgb_camera_optical_frame"/>
+			<child link="${name}_color_optical_frame"/>
+			<origin xyz="0 0 0" rpy="0 0 0"/>
+		</joint>
 		<!-- Depth/Stereo camera frames -->
 		<link name="${name}_stereo_camera_frame"/>
