Commit message: feat(perception): этап 0 ADR-0130 — chrony между Pi, фрейм микрофона в URDF, инструменты замера DOA и нагрузки (ADR-0137)
Дочерний ADR-0137 этапа 0 ADR-0130 §7. Робота в этой сессии нет:
инструменты и фрейм готовы, ни одного замера на роботе не сделано,
статус ADR — Proposed.

- scripts/maintenance/setup_chrony.sh: chrony на хостах обоих Pi,
  --role main (внешние пулы + allow 10.1.1.0/24 + local stratum 10) |
  vision (server 10.1.1.10 iburst prefer — eth0 Main Pi по проводу, а не
  Wi-Fi 10.1.1.20; переопределяется --server); --check печатает
  «chrony_check … verdict=PASS|FAIL», FAIL при |offset| > 5 мс или чужом
  источнике; отключает systemd-timesyncd (один писатель времени на Pi).
- scripts/maintenance/sync_time.sh: помечен устаревшим с ADR-0137; если
  chrony активен — timesyncd не трогает и делегирует setup_chrony.sh
  --check (деплой L-Deploy and Verify продолжает его звать).
- rob_box.xacro: фрейм mic_array_link (fixed к base_link, xyz 0 0 0.46,
  rpy 0 0 0) — ЗАГЛУШКА: физическое положение ReSpeaker нигде не
  задокументировано, измерить (ADR-0137 §4 в.1–2).
- scripts/maintenance/measure_doa.py: замер точности DOA по известным
  углам только при VAD, CSV + p50/p95 + вердикт ≤15° (ADR-0130 Q17).
- scripts/maintenance/measure_load.sh: CPU/MEM по контейнерам, load1,
  температура, NPU-снимок через hailortcli если есть (в образе
  vision-hailo его нет — честно «NPU metric unavailable»).
- tests/unit/maintenance/: 57 тестов на чистые функции и CLI скриптов
  (папка в CI не подключена — как и соседний тест там же).

Найдено попутно (ADR-0137 §1): audio_node.py:1035 зовёт
respeaker.get_direction(), у ReSpeakerInterface есть только get_doa();
AttributeError глотается except Exception: pass → /audio/direction по коду
не публикуется никогда. Посылка ADR-0130 §1.3 «публикуется всегда» неверна;
фикс — отдельным коммитом.

Проверка (raw в PR): pytest tests/unit/maintenance — 57 passed, 1 skipped
(root в песочнице); bash -n ×3 ok; shellcheck 0.11.0 ×3 rc=0; flake8 с
флагами CI (max-line-length=120, ignore E501) rc=0; xacro → URDF
well-formed, links 18→19, joints 17→18, цепочка mic_array_link ← base_link.
Лабораторный прогон chrony 4.5 в песочнице: два chronyd -x на loopback,
--check role=vision offset_ms=0.005 verdict=PASS rc=0; неверный источник
→ FAIL rc=2; chronyd мёртв → rc=3. systemctl-шаги в песочнице не проверены.

НЕ проверено: установка на Pi, реальный offset Vision↔Main, поведение
после ребута и под деплоем, замер DOA (заблокирован багом get_direction),
docker stats/vcgencmd/hailortcli на живом Pi, TF нового фрейма у
robot_state_publisher, физическое положение микрофона.

Refs #2995.

Co-Authored-By: Claude Fable 5.1 <noreply@anthropic.com>
Claude-Session: https://claude.ai/code/session_01685NVgWwrfqXMGhw2DEa26

File: src/rob_box_description/urdf/rob_box.xacro (robot description, xacro)
@@ -11,4 +11,12 @@
 	<xacro:property name="rocker_mass" value="3"/>
 	<xacro:property name="base_mass" value="62.64527022934752"/>  <!-- От Fusion 360: 62.65 кг -->
+	<!-- Микрофонный массив ReSpeaker USB Mic Array v2.0 (ADR-0130 §2.9, ADR-0137 §2.2). -->
+	<!-- ЗАГЛУШКА: физическое положение нигде не задокументировано и не измерено.   -->
+	<!-- z = 0.46 м над base_link — «на уровне камер» (OAK-D 0.4595, лидар 0.4765),  -->
+	<!-- x = y = 0 — центр корпуса. Измерить рулеткой и заменить (ADR-0137 §4, в.1). -->
+	<!-- yaw: ось X фрейма = направление, в котором прошивка отдаёт DOAANGLE = 0°;    -->
+	<!-- знак отсчёта (по/против часовой) и yaw — из замера measure_doa.py (§4, в.2). -->
+	<xacro:property name="mic_array_xyz" value="0 0 0.46"/>
+	<xacro:property name="mic_array_rpy" value="0 0 0"/>
 	<!-- base_footprint - корневой фрейм робота на уровне пола -->
 	<!-- Используется как reference frame в соответствии с REP-120 -->
@@ -321,4 +329,12 @@
 	<!-- Поворот на 90° по часовой стрелке вокруг Y (pitch=-90°) для правильной ориентации -->
 	<xacro:usb_camera name="ceiling_camera" parent_link="base_link" origin_xyz="-0.170663 0.065 0.4615" origin_rpy="0 0 0"/>
+	<!-- Микрофонный массив: только фрейм (без меша). Центр массива, Z вверх.     -->
+	<!-- Потребитель — азимут DOA → трек (ADR-0130 §2.9, этап 5). ЗАГЛУШКА, см. выше. -->
+	<link name="mic_array_link"/>
+	<joint name="mic_array_joint" type="fixed">
+		<parent link="base_link"/>
+		<child link="mic_array_link"/>
+		<origin xyz="${mic_array_xyz}" rpy="${mic_array_rpy}"/>
+	</joint>
 	<!-- ros2_control Hardware Interface - VESC Nexus -->
 	<xacro:include filename="rob_box_ros2_control.xacro"/>

Commit message: fix(description): положение фрейма mic_array_link со слов владельца (ADR-0137 §2.2)
Владелец 28.09.2026: ReSpeaker стоит на высоте лидара, чуть левее, почти
симметрично потолочной камере. Заглушка 0 0 0.46 заменена на
-0.1707 -0.06 0.4765: z лидара (0.4765), x лидара и потолочной камеры
(-0.1707), по борту зеркально потолочной камере (y=+0.065): «левее»
трактовано как «слева при взгляде на робота спереди» → правый борт, y<0.
Знак y требует подтверждения, рулеткой не измерено; на азимут DOA не
влияет — yaw и знак отсчёта калибруются measure_doa.py (§2.3).
ADR-0137: TL;DR, F4, §2.2, §3, §4 в.1 обновлены.

Проверка: xacro → origin xyz="-0.1707 -0.06 0.4765" у mic_array_joint;
pytest tests/unit/maintenance — 57 passed, 1 skipped.

Co-Authored-By: Claude Fable 5.1 <noreply@anthropic.com>
Claude-Session: https://claude.ai/code/session_01685NVgWwrfqXMGhw2DEa26

File: src/rob_box_description/urdf/rob_box.xacro (robot description, xacro)
@@ -12,10 +12,11 @@
 	<xacro:property name="base_mass" value="62.64527022934752"/>  <!-- От Fusion 360: 62.65 кг -->
 	<!-- Микрофонный массив ReSpeaker USB Mic Array v2.0 (ADR-0130 §2.9, ADR-0137 §2.2). -->
-	<!-- ЗАГЛУШКА: физическое положение нигде не задокументировано и не измерено.   -->
-	<!-- z = 0.46 м над base_link — «на уровне камер» (OAK-D 0.4595, лидар 0.4765),  -->
-	<!-- x = y = 0 — центр корпуса. Измерить рулеткой и заменить (ADR-0137 §4, в.1). -->
+	<!-- Положение со слов владельца (28.09.2026): на высоте лидара (z=0.4765), в той же  -->
+	<!-- плоскости x, что лидар и потолочная камера (x≈-0.1707), по борту — почти зеркально -->
+	<!-- потолочной камере (y=+0.065): «чуть левее», если смотреть на робота спереди, т.е.  -->
+	<!-- правый борт робота, y≈-0.06. Рулеткой не измерено — уточнить (ADR-0137 §4, в.1). -->
 	<!-- yaw: ось X фрейма = направление, в котором прошивка отдаёт DOAANGLE = 0°;    -->
 	<!-- знак отсчёта (по/против часовой) и yaw — из замера measure_doa.py (§4, в.2). -->
-	<xacro:property name="mic_array_xyz" value="0 0 0.46"/>
+	<xacro:property name="mic_array_xyz" value="-0.1707 -0.06 0.4765"/>
 	<xacro:property name="mic_array_rpy" value="0 0 0"/>
 	<!-- base_footprint - корневой фрейм робота на уровне пола -->
@@ -330,5 +331,5 @@
 	<xacro:usb_camera name="ceiling_camera" parent_link="base_link" origin_xyz="-0.170663 0.065 0.4615" origin_rpy="0 0 0"/>
 	<!-- Микрофонный массив: только фрейм (без меша). Центр массива, Z вверх.     -->
-	<!-- Потребитель — азимут DOA → трек (ADR-0130 §2.9, этап 5). ЗАГЛУШКА, см. выше. -->
+	<!-- Потребитель — азимут DOA → трек (ADR-0130 §2.9, этап 5). Положение — см. выше. -->
 	<link name="mic_array_link"/>
 	<joint name="mic_array_joint" type="fixed">

Commit message: fix(description): mic_array_link на том же борту, что потолочная камера; факт про ориентацию камеры (ADR-0137)
Уточнение владельца 28.09.2026: при взгляде на робота лицом к лицу и
потолочная камера, и ReSpeaker — справа, то есть левый борт робота (+y);
камера на y=+0.065, микрофон чуть ближе к центру → mic_array_xyz =
-0.1707 0.05 0.4765 (прежняя трактовка y<0 была неверна). Рулеткой не
измерено.

Попутно зафиксировано в ADR-0137 §1 (F4a): потолочная камера физически
смотрит линзой в потолок, а в rob_box.xacro:352 origin_rpy="0 0 0"
(фрейм «вперёд»). Это закрывает открытый вопрос ADR-0130 §8 п.2 (камера
в распознавании людей не участвует); правка ориентации фрейма — отдельной
карточкой, вне этапа 0.

Проверка: xacro → origin xyz="-0.1707 0.05 0.4765" у mic_array_joint.

Co-Authored-By: Claude Fable 5.1 <noreply@anthropic.com>
Claude-Session: https://claude.ai/code/session_01685NVgWwrfqXMGhw2DEa26

File: src/rob_box_description/urdf/rob_box.xacro (robot description, xacro)
@@ -13,10 +13,10 @@
 	<!-- Микрофонный массив ReSpeaker USB Mic Array v2.0 (ADR-0130 §2.9, ADR-0137 §2.2). -->
 	<!-- Положение со слов владельца (28.09.2026): на высоте лидара (z=0.4765), в той же  -->
-	<!-- плоскости x, что лидар и потолочная камера (x≈-0.1707), по борту — почти зеркально -->
-	<!-- потолочной камере (y=+0.065): «чуть левее», если смотреть на робота спереди, т.е.  -->
-	<!-- правый борт робота, y≈-0.06. Рулеткой не измерено — уточнить (ADR-0137 §4, в.1). -->
+	<!-- плоскости x, что лидар и потолочная камера (x≈-0.1707), на ТОМ ЖЕ борту, что и   -->
+	<!-- потолочная камера (y=+0.065, левый борт робота = справа при взгляде на робота     -->
+	<!-- лицом к лицу), чуть ближе к центру: y≈+0.05. Рулеткой не измерено (ADR-0137 §4, в.1). -->
 	<!-- yaw: ось X фрейма = направление, в котором прошивка отдаёт DOAANGLE = 0°;    -->
 	<!-- знак отсчёта (по/против часовой) и yaw — из замера measure_doa.py (§4, в.2). -->
-	<xacro:property name="mic_array_xyz" value="-0.1707 -0.06 0.4765"/>
+	<xacro:property name="mic_array_xyz" value="-0.1707 0.05 0.4765"/>
 	<xacro:property name="mic_array_rpy" value="0 0 0"/>
 	<!-- base_footprint - корневой фрейм робота на уровне пола -->
