Commit message: feat(perception): ADR-0130 этапы 0–1 — Observation.msg + глубина OAK-D, chrony/фрейм микрофона, фикс /audio/direction, ADR-0139 (#3124)
* docs(adr): восстановить контракт face→voice hint как ADR-0139, починить ссылки ADR-0135 (#3024, #3040)

PR #3040 ссылался на «ADR-0135», но файла такого ADR в истории нет:
номер 0135 занят параллельным PR #3031 (face-picker Quest). Контракт
face-hint (FaceSignal/FaceObservation, полосы 0.78/0.65, окно 30 с,
буфер 8, флаг face_voice_hint.enabled) оставался без документа, ссылки
в коде вели в никуда (ADR-AF-0030 — нумерация ADR как SOT).

- docs/adr/0139-face-voice-hint-identity-seam.md: текст реконструирован
  по identity/base.py, dialogue_node.py, обоим dialogue_node.yaml и
  acceptance-тесту; секции совпадают с номерами, на которые ссылается
  код (§2.1–§2.6, §3, §5.2, §6.1). Статус — Accepted (реализовано
  PR #3040), с явной пометкой о реконструкции.
- ADR-0135 → ADR-0139 в комментариях/докстрингах/логах identity/base.py,
  dialogue_node.py, обоих dialogue_node.yaml и теста #3024. Ссылки на
  настоящий ADR-0135 (face_card.py, face_collage.py) не тронуты.
- Связь с ADR-0130 §2.6 путь 2: hint — предшественник v2.0-улики
  «два канала согласны».

Проверка: test_issue_3024_face_hint_suppresses_voice_recheck.py — 9 passed;
rob_box_harness -k "identity or face" — 18 passed;
grep -rn "ADR-0135" src docker → только face_card.py:548 и face_collage.py:5.
test_yaml_param_consistency.py: 2 failed / 20 passed — те же 2 падения на
чистом origin/develop (voice_preset не объявлен, нет voice_assistant.yaml),
к этому коммиту не относятся.

Co-Authored-By: Claude Fable 5.1 <noreply@anthropic.com>
Claude-Session: https://claude.ai/code/session_01685NVgWwrfqXMGhw2DEa26

* feat(perception): этап 1 ADR-0130 — Observation.msg, глубина OAK-D через «Взгляд», distance_m вместо −1 (ADR-0138)

Дочерний ADR-0138 этапа 1 ADR-0130 §7: наблюдения датчика с геометрией,
без имён и без собственного id личности (инварианты §5.1 п.1, п.5, п.7).

- rob_box_perception_msgs/msg/Observation.msg: header (stamp и frame_id
  КАДРА, optical frame камеры), source, class_name person|face, bbox в
  пикселях + размер кадра, position (Point, NaN при отказе глубины),
  distance_m (−1 при отказе), position_valid + position_status (9 честных
  статусов), position_stddev_m, candidate_id + candidate_similarity.
  VisionEvent.msg помечен deprecated (поля не менялись).
- gaze.py: Frame получает depth_mm / intrinsics / depth_status; OakDSource
  дополнительно подписан на /camera/camera/depth/image_rect_raw и
  /camera/camera/color/camera_info, связывание по ближайшему stamp
  (буфер 8, допуск 0.15 с), повторное связывание при опоздавшей глубине.
  TF и message_filters не используются: в base_link/map переводит трекер
  на Main Pi (этап 2, ADR-0130 §2.11).
- observation_geometry.py: чистый модуль без ROS — медиана глубины по
  центральным 50 % бокса с отсечением по MAD, перевод через K, stddev по
  инлаерам; build_observation, OBSERVATION_FIELDS, словарь статусов.
- vision_hailo_node.py: кадр фиксируется один раз в _tick; VisionEvent
  .distance_m берётся из той же оценки; Observation публикуется на
  observation_topic (default /perception/observations) для person/face из
  реального кадра, stub-события не публикуются. Новые параметры
  observation_topic, depth_enabled, depth_sync_tolerance_sec прокинуты в
  launch_factory, hailo_models.yaml и оба start-скрипта.

Проверка (raw в PR): pytest src/rob_box_perception/test/unit
(--ignore core) — 374 passed, 33 skipped (база 317/32; +57 тестов,
1 skip — паритет с сгенерированным msg требует colcon). flake8
(max-line-length=99) по 7 новым/изменённым py — rc=0. bash -n обоих
start-скриптов — ok. Мутационная проверка: без заполнения distance_m —
2 failed; без повторного связывания глубины — 1 failed.

Архитектурный аудит (tools/architecture_audit.py + findings) до/после:
78 → 78 находок, new [] gone []; inventory: +1 py-файл, +1 класс
(PositionEstimate), +4 тест-файла. Ограничение инструмента: топик задан
параметром observation_topic, статический скан его не видит (как и
/vision/hailo/events). На runtime-аудите ожидаются dead_output и
multiple_writers для /perception/observations до трекера этапа 2 —
записано в ADR-0138 §3 как временное.

НЕ проверено: colcon build msg-пакета, тесты под настоящим rclpy, работа
на роботе (реальный depth-топик и его encoding при i_low_bandwidth,
frame_id, CPU Vision Pi, доставка через Zenoh). e2e не прогонялся.

Refs #2995 (этап 4 стоит на этапах 0–3).

Co-Authored-By: Claude Fable 5.1 <noreply@anthropic.com>
Claude-Session: https://claude.ai/code/session_01685NVgWwrfqXMGhw2DEa26

* feat(perception): этап 0 ADR-0130 — chrony между Pi, фрейм микрофона в URDF, инструменты замера DOA и нагрузки (ADR-0137)

Дочерний ADR-0137 этапа 0 ADR-0130 §7. Робота в этой сессии нет:
инструменты и фрейм готовы, ни одного замера на роботе не сделано,
статус ADR — Proposed.

- scripts/maintenance/setup_chrony.sh: chrony на хостах обоих Pi,
  --role main (внешние пулы + allow 10.1.1.0/24 + local stratum 10) |
  vision (server 10.1.1.10 iburst prefer — eth0 Main Pi по проводу, а не
  Wi-Fi 10.1.1.20; переопределяется --server); --check печатает
  «chrony_check … verdict=PASS|FAIL», FAIL при |offset| > 5 мс или чужом
  источнике; отключает systemd-timesyncd (один писатель времени на Pi).
- scripts/maintenance/sync_time.sh: помечен устаревшим с ADR-0137; если
  chrony активен — timesyncd не трогает и делегирует setup_chrony.sh
  --check (деплой L-Deploy and Verify продолжает его звать).
- rob_box.xacro: фрейм mic_array_link (fixed к base_link, xyz 0 0 0.46,
  rpy 0 0 0) — ЗАГЛУШКА: физическое положение ReSpeaker нигде не
  задокументировано, измерить (ADR-0137 §4 в.1–2).
- scripts/maintenance/measure_doa.py: замер точности DOA по известным
  углам только при VAD, CSV + p50/p95 + вердикт ≤15° (ADR-0130 Q17).
- scripts/maintenance/measure_load.sh: CPU/MEM по контейнерам, load1,
  температура, NPU-снимок через hailortcli если есть (в образе
  vision-hailo его нет — честно «NPU metric unavailable»).
- tests/unit/maintenance/: 57 тестов на чистые функции и CLI скриптов
  (папка в CI не подключена — как и соседний тест там же).

Найдено попутно (ADR-0137 §1): audio_node.py:1035 зовёт
respeaker.get_direction(), у ReSpeakerInterface есть только get_doa();
AttributeError глотается except Exception: pass → /audio/direction по коду
не публикуется никогда. Посылка ADR-0130 §1.3 «публикуется всегда» неверна;
фикс — отдельным коммитом.

Проверка (raw в PR): pytest tests/unit/maintenance — 57 passed, 1 skipped
(root в песочнице); bash -n ×3 ok; shellcheck 0.11.0 ×3 rc=0; flake8 с
флагами CI (max-line-length=120, ignore E501) rc=0; xacro → URDF
well-formed, links 18→19, joints 17→18, цепочка mic_array_link ← base_link.
Лабораторный прогон chrony 4.5 в песочнице: два chronyd -x на loopback,
--check role=vision offset_ms=0.005 verdict=PASS rc=0; неверный источник
→ FAIL rc=2; chronyd мёртв → rc=3. systemctl-шаги в песочнице не проверены.

НЕ проверено: установка на Pi, реальный offset Vision↔Main, поведение
после ребута и под деплоем, замер DOA (заблокирован багом get_direction),
docker stats/vcgencmd/hailortcli на живом Pi, TF нового фрейма у
robot_state_publisher, физическое положение микрофона.

Refs #2995.

Co-Authored-By: Claude Fable 5.1 <noreply@anthropic.com>
Claude-Session: https://claude.ai/code/session_01685NVgWwrfqXMGhw2DEa26

* fix(lint): allowlist швов этапа 1 ADR-0130 для seam_without_consumer (ADR-0138 §3)

Гейт G-Lint Code (scripts/lint/seam_without_consumer.py, ADR-0021) падал
на коммите e0f4e359: «FAIL — 3 new seam(s) without consumer»:
  /perception/observations         (vision_hailo_node.py:304, publisher)
  /camera/camera/color/camera_info (gaze.py:448, subscriber)
  /camera/camera/depth/image_rect_raw (gaze.py:445, subscriber)

- seam_allowlist.json: два camera-топика публикует внешний драйвер
  depthai_ros_driver (контейнер oak-d, C++, не в src/), потребитель —
  gaze.OakDSource (ADR-0138 §2.4); /perception/observations помечен
  ВРЕМЕННО до трекера этапа 2 ADR-0130 (запись удалить в PR этапа 2).
  seam_baseline.json не тронут.
- ADR-0138 §3 и §7 п.6: уточнено, что разрыв есть только у
  tools/architecture_audit.py (литеральные имена), а seam-линтер шов
  видит через резолв параметра.

Проверка: python scripts/lint/seam_without_consumer.py →
«OK — no new seams without consumer» (rc=0);
python -m unittest scripts.lint.test_seam_without_consumer → Ran 48 tests, OK.
Сам CI-run не запускался — «CI зелёный» не утверждается.

Co-Authored-By: Claude Fable 5.1 <noreply@anthropic.com>
Claude-Session: https://claude.ai/code/session_01685NVgWwrfqXMGhw2DEa26

* fix(voice): /audio/direction никогда не публиковался — get_direction() вместо get_doa()

audio_node.py:1035 звал self.respeaker.get_direction(), но у
ReSpeakerInterface (utils/respeaker_interface.py:209) есть только
get_doa() -> Optional[int]. AttributeError глотался «except Exception:
pass» (комментарий «pipe error»), поэтому DOA не публиковался никогда.
git log -S"def get_direction" — пусто: метода не существовало ни в одной
ревизии. Существующие тесты подменяли respeaker через MagicMock() без
spec и дыру не видели. Посылка ADR-0130 §1.3 «/audio/direction
публикуется всегда» по коду была неверна; блокировало замер DOA этапа 0
(ADR-0137 §1, §2.3).

- get_direction() → get_doa().
- Вместо тихого pass: AttributeError/TypeError — ошибка кода, ERROR с
  exc_info; usb.core.USBError/OSError — WARN; оба через уже существующий
  троттлинг _vad_doa_last_warn_ns / _vad_doa_warn_period_ns (60 с,
  issue #1125), новых механизмов нет. import usb.core — pyusb уже в
  requirements.txt и импортируется respeaker_interface на уровне модуля.
- test_audio_node_echo.py: TestDirectionPublishUsesGetDoa —
  MagicMock(spec=настоящий ReSpeakerInterface): get_doa()=123 →
  publish(Int32 123) ровно один раз; get_doa()=None → без публикации.
  Мёртвый мок get_direction в соседнем тесте заменён на get_doa.

Проверка (raw в PR): мутационно — с get_direction в проде новый тест
FAIL («Expected 'publish' to have been called once. Called 0 times»);
после фикса — 2 passed. test_audio_node_echo + test_issue_2701 +
unit/test_audio_node_no_bare_except: 62 passed. Весь src/rob_box_voice/test
(без test_audio_node.py, который падает на import rclpy и до правок):
3971 passed, 39 skipped. flake8: новых находок нет (pre-existing E501/E261/
F841 на месте).

НЕ проверено на роботе с реальным ReSpeaker. Осталось: 4 мёртвых мока
get_direction в test_issue_2701_audio_watchdog.py (тесты не ломают).

Co-Authored-By: Claude Fable 5.1 <noreply@anthropic.com>
Claude-Session: https://claude.ai/code/session_01685NVgWwrfqXMGhw2DEa26

* fix(description): положение фрейма mic_array_link со слов владельца (ADR-0137 §2.2)

Владелец 28.09.2026: ReSpeaker стоит на высоте лидара, чуть левее, почти
симметрично потолочной камере. Заглушка 0 0 0.46 заменена на
-0.1707 -0.06 0.4765: z лидара (0.4765), x лидара и потолочной камеры
(-0.1707), по борту зеркально потолочной камере (y=+0.065): «левее»
трактовано как «слева при взгляде на робота спереди» → правый борт, y<0.
Знак y требует подтверждения, рулеткой не измерено; на азимут DOA не
влияет — yaw и знак отсчёта калибруются measure_doa.py (§2.3).
ADR-0137: TL;DR, F4, §2.2, §3, §4 в.1 обновлены.

Проверка: xacro → origin xyz="-0.1707 -0.06 0.4765" у mic_array_joint;
pytest tests/unit/maintenance — 57 passed, 1 skipped.

Co-Authored-By: Claude Fable 5.1 <noreply@anthropic.com>
Claude-Session: https://claude.ai/code/session_01685NVgWwrfqXMGhw2DEa26

* fix(description): mic_array_link на том же борту, что потолочная камера; факт про ориентацию камеры (ADR-0137)

Уточнение владельца 28.09.2026: при взгляде на робота лицом к лицу и
потолочная камера, и ReSpeaker — справа, то есть левый борт робота (+y);
камера на y=+0.065, микрофон чуть ближе к центру → mic_array_xyz =
-0.1707 0.05 0.4765 (прежняя трактовка y<0 была неверна). Рулеткой не
измерено.

Попутно зафиксировано в ADR-0137 §1 (F4a): потолочная камера физически
смотрит линзой в потолок, а в rob_box.xacro:352 origin_rpy="0 0 0"
(фрейм «вперёд»). Это закрывает открытый вопрос ADR-0130 §8 п.2 (камера
в распознавании людей не участвует); правка ориентации фрейма — отдельной
карточкой, вне этапа 0.

Проверка: xacro → origin xyz="-0.1707 0.05 0.4765" у mic_array_joint.

Co-Authored-By: Claude Fable 5.1 <noreply@anthropic.com>
Claude-Session: https://claude.ai/code/session_01685NVgWwrfqXMGhw2DEa26

* refactor(voice): вынести чтение DOA из check_vad_and_doa — CC-budget гейт (ADR-0021)

CI G-Lint Code (run 36446937421, job 109011564926) упал:
«[FAIL] audio_node.py:AudioNode.check_vad_and_doa CC=24 grew past
baseline 19» — фикс dd60d25d добавил ветки обработки ошибок DOA.

- DOA-блок (get_doa, публикация, два except) вынесен в
  _read_and_publish_doa(); имя вне паттернов _publish_*/_on_* seam-линтера,
  вызывается из check_vad_and_doa.
- троттлинг предупреждений — один helper _vad_doa_warn_throttle_ready()
  вместо трёх одинаковых условий (включая старый общий except).
  cc_budget_baseline.json не тронут.

Проверка: python scripts/lint/cc_budget.py → check_vad_and_doa CC=16
(baseline 19), «OK — no new CC violations»; seam_without_consumer → OK;
cc_budget_refs rc=0; pytest test_audio_node_echo + test_issue_2701 +
unit/test_audio_node_no_bare_except + unit/test_audio_node_bytecode —
70 passed. Поведение снаружи не менялось, оба DOA-теста зелёные без
правок. flake8: только прежние E501/E261/F841, новых нет.

Co-Authored-By: Claude Fable 5.1 <noreply@anthropic.com>
Claude-Session: https://claude.ai/code/session_01685NVgWwrfqXMGhw2DEa26

---------

Co-authored-by: Claude <noreply@anthropic.com>

File: src/rob_box_description/urdf/rob_box.xacro (robot description, xacro)
@@ -11,4 +11,13 @@
 	<xacro:property name="rocker_mass" value="3"/>
 	<xacro:property name="base_mass" value="62.64527022934752"/>  <!-- От Fusion 360: 62.65 кг -->
+	<!-- Микрофонный массив ReSpeaker USB Mic Array v2.0 (ADR-0130 §2.9, ADR-0137 §2.2). -->
+	<!-- Положение со слов владельца (28.09.2026): на высоте лидара (z=0.4765), в той же  -->
+	<!-- плоскости x, что лидар и потолочная камера (x≈-0.1707), на ТОМ ЖЕ борту, что и   -->
+	<!-- потолочная камера (y=+0.065, левый борт робота = справа при взгляде на робота     -->
+	<!-- лицом к лицу), чуть ближе к центру: y≈+0.05. Рулеткой не измерено (ADR-0137 §4, в.1). -->
+	<!-- yaw: ось X фрейма = направление, в котором прошивка отдаёт DOAANGLE = 0°;    -->
+	<!-- знак отсчёта (по/против часовой) и yaw — из замера measure_doa.py (§4, в.2). -->
+	<xacro:property name="mic_array_xyz" value="-0.1707 0.05 0.4765"/>
+	<xacro:property name="mic_array_rpy" value="0 0 0"/>
 	<!-- base_footprint - корневой фрейм робота на уровне пола -->
 	<!-- Используется как reference frame в соответствии с REP-120 -->
@@ -321,4 +330,12 @@
 	<!-- Поворот на 90° по часовой стрелке вокруг Y (pitch=-90°) для правильной ориентации -->
 	<xacro:usb_camera name="ceiling_camera" parent_link="base_link" origin_xyz="-0.170663 0.065 0.4615" origin_rpy="0 0 0"/>
+	<!-- Микрофонный массив: только фрейм (без меша). Центр массива, Z вверх.     -->
+	<!-- Потребитель — азимут DOA → трек (ADR-0130 §2.9, этап 5). Положение — см. выше. -->
+	<link name="mic_array_link"/>
+	<joint name="mic_array_joint" type="fixed">
+		<parent link="base_link"/>
+		<child link="mic_array_link"/>
+		<origin xyz="${mic_array_xyz}" rpy="${mic_array_rpy}"/>
+	</joint>
 	<!-- ros2_control Hardware Interface - VESC Nexus -->
 	<xacro:include filename="rob_box_ros2_control.xacro"/>
