Commit message: fix(urdf): Update inertial properties and joint origins for improved robot model accuracy

File: src/rob_box_description/URDF_EXPORT/urdf/URDF_ROBBOX.xacro (robot description, xacro)
@@ -6,7 +6,7 @@
 <link name="base_link">
   <inertial>
-    <origin xyz="-2.4090750286344156e-05 0.025488169162562517 0.14529190576177464" rpy="0 0 0"/>
-    <mass value="62.64527022934752"/>
-    <inertia ixx="2.829827" iyy="1.926172" izz="3.653023" ixy="-0.001791" iyz="-0.302171" ixz="-0.001655"/>
+    <origin xyz="-0.025488169162561854 -2.4090750285970683e-05 0.14529190576177384" rpy="0 0 0"/>
+    <mass value="62.6452702293474"/>
+    <inertia ixx="1.926172" iyy="2.829827" izz="3.653023" ixy="0.001791" iyz="-0.001655" ixz="0.302171"/>
   </inertial>
   <visual>
@@ -26,10 +26,10 @@
 <link name="camera_rpi_1">
   <inertial>
-    <origin xyz="-5.712518555411883e-09 -3.993788821321509e-07 0.008386121687044445" rpy="0 0 0"/>
-    <mass value="0.029114258669862975"/>
-    <inertia ixx="2e-06" iyy="2e-06" izz="1e-06" ixy="0.0" iyz="0.0" ixz="-0.0"/>
-  </inertial>
-  <visual>
-    <origin xyz="-0.065 -0.170663 -0.4615" rpy="0 0 0"/>
+    <origin xyz="3.993788821321509e-07 -5.712548975522758e-09 0.008386121687044445" rpy="0 0 0"/>
+    <mass value="0.02911425866986295"/>
+    <inertia ixx="2e-06" iyy="2e-06" izz="1e-06" ixy="-0.0" iyz="-0.0" ixz="0.0"/>
+  </inertial>
+  <visual>
+    <origin xyz="0.170663 -0.065 -0.4615" rpy="0 0 0"/>
     <geometry>
       <mesh filename="package://URDF_ROBBOX_description/meshes/camera_rpi_1.stl" scale="0.001 0.001 0.001"/>
@@ -38,5 +38,5 @@
   </visual>
   <collision>
-    <origin xyz="-0.065 -0.170663 -0.4615" rpy="0 0 0"/>
+    <origin xyz="0.170663 -0.065 -0.4615" rpy="0 0 0"/>
     <geometry>
       <mesh filename="package://URDF_ROBBOX_description/meshes/camera_rpi_1.stl" scale="0.001 0.001 0.001"/>
@@ -46,10 +46,10 @@
 <link name="lidar_1">
   <inertial>
-    <origin xyz="-4.053001291838554e-07 2.840693373307168e-07 0.01805000000000001" rpy="0 0 0"/>
+    <origin xyz="-2.840693373307168e-07 -4.053001292181704e-07 0.01805000000000001" rpy="0 0 0"/>
     <mass value="0.6018294382769799"/>
-    <inertia ixx="0.000167" iyy="0.000167" izz="0.000203" ixy="0.0" iyz="-0.0" ixz="0.0"/>
-  </inertial>
-  <visual>
-    <origin xyz="0.000331 -0.170806 -0.4765" rpy="0 0 0"/>
+    <inertia ixx="0.000167" iyy="0.000167" izz="0.000203" ixy="0.0" iyz="0.0" ixz="0.0"/>
+  </inertial>
+  <visual>
+    <origin xyz="0.170806 0.000331 -0.4765" rpy="0 0 0"/>
     <geometry>
       <mesh filename="package://URDF_ROBBOX_description/meshes/lidar_1.stl" scale="0.001 0.001 0.001"/>
@@ -58,5 +58,5 @@
   </visual>
   <collision>
-    <origin xyz="0.000331 -0.170806 -0.4765" rpy="0 0 0"/>
+    <origin xyz="0.170806 0.000331 -0.4765" rpy="0 0 0"/>
     <geometry>
       <mesh filename="package://URDF_ROBBOX_description/meshes/lidar_1.stl" scale="0.001 0.001 0.001"/>
@@ -66,10 +66,10 @@
 <link name="camera_oak_1">
   <inertial>
-    <origin xyz="3.86015228183602e-07 -0.008750436983790896 -0.014999999999999791" rpy="0 0 0"/>
-    <mass value="0.3500314999999997"/>
-    <inertia ixx="3.2e-05" iyy="0.000264" izz="0.00025" ixy="-0.0" iyz="0.0" ixz="0.0"/>
-  </inertial>
-  <visual>
-    <origin xyz="0.000238 -0.115772 -0.4595" rpy="0 0 0"/>
+    <origin xyz="0.008750436983790896 0.015000386015228177 2.220446049250313e-16" rpy="0 0 0"/>
+    <mass value="0.3500314999999998"/>
+    <inertia ixx="0.000264" iyy="3.2e-05" izz="0.00025" ixy="0.0" iyz="0.0" ixz="-0.0"/>
+  </inertial>
+  <visual>
+    <origin xyz="0.115772 0.000238 -0.4595" rpy="0 0 0"/>
     <geometry>
       <mesh filename="package://URDF_ROBBOX_description/meshes/camera_oak_1.stl" scale="0.001 0.001 0.001"/>
@@ -78,5 +78,5 @@
   </visual>
   <collision>
-    <origin xyz="0.000238 -0.115772 -0.4595" rpy="0 0 0"/>
+    <origin xyz="0.115772 0.000238 -0.4595" rpy="0 0 0"/>
     <geometry>
       <mesh filename="package://URDF_ROBBOX_description/meshes/camera_oak_1.stl" scale="0.001 0.001 0.001"/>
@@ -86,10 +86,10 @@
 <link name="wheel_rear_left_1">
   <inertial>
-    <origin xyz="0.037500000000000006 4.886100668233251e-07 -3.196217084333597e-07" rpy="0 0 0"/>
-    <mass value="21.68159743475603"/>
-    <inertia ixx="0.129466" iyy="0.073667" izz="0.073667" ixy="0.0" iyz="0.0" ixz="0.0"/>
-  </inertial>
-  <visual>
-    <origin xyz="-0.195 -0.143797 -0.028767" rpy="0 0 0"/>
+    <origin xyz="-4.886100668233251e-07 0.03749999999999995 -3.196217084333597e-07" rpy="0 0 0"/>
+    <mass value="21.681597434756032"/>
+    <inertia ixx="0.073667" iyy="0.129466" izz="0.073667" ixy="0.0" iyz="0.0" ixz="0.0"/>
+  </inertial>
+  <visual>
+    <origin xyz="0.143797 -0.195 -0.028767" rpy="0 0 0"/>
     <geometry>
       <mesh filename="package://URDF_ROBBOX_description/meshes/wheel_rear_left_1.stl" scale="0.001 0.001 0.001"/>
@@ -98,5 +98,5 @@
   </visual>
   <collision>
-    <origin xyz="-0.195 -0.143797 -0.028767" rpy="0 0 0"/>
+    <origin xyz="0.143797 -0.195 -0.028767" rpy="0 0 0"/>
     <geometry>
       <mesh filename="package://URDF_ROBBOX_description/meshes/wheel_rear_left_1.stl" scale="0.001 0.001 0.001"/>
@@ -106,10 +106,10 @@
 <link name="wheel_front_left_1">
   <inertial>
-    <origin xyz="0.037500000000000006 -3.689894347569389e-07 -2.7755575615628914e-17" rpy="0 0 0"/>
+    <origin xyz="3.689894347569389e-07 0.03750000000000006 -3.469446951953614e-18" rpy="0 0 0"/>
     <mass value="21.68159743475604"/>
-    <inertia ixx="0.129466" iyy="0.073667" izz="0.073667" ixy="0.0" iyz="-0.0" ixz="0.0"/>
-  </inertial>
-  <visual>
-    <origin xyz="-0.195 0.145731 -0.0289" rpy="0 0 0"/>
+    <inertia ixx="0.073667" iyy="0.129466" izz="0.073667" ixy="-0.0" iyz="0.0" ixz="0.0"/>
+  </inertial>
+  <visual>
+    <origin xyz="-0.145731 -0.195 -0.0289" rpy="0 0 0"/>
     <geometry>
       <mesh filename="package://URDF_ROBBOX_description/meshes/wheel_front_left_1.stl" scale="0.001 0.001 0.001"/>
@@ -118,5 +118,5 @@
   </visual>
   <collision>
-    <origin xyz="-0.195 0.145731 -0.0289" rpy="0 0 0"/>
+    <origin xyz="-0.145731 -0.195 -0.0289" rpy="0 0 0"/>
     <geometry>
       <mesh filename="package://URDF_ROBBOX_description/meshes/wheel_front_left_1.stl" scale="0.001 0.001 0.001"/>
@@ -126,10 +126,10 @@
 <link name="wheel_front_right_1">
   <inertial>
-    <origin xyz="-0.037500289005600596 3.689894347569389e-07 -1.3877787807814457e-17" rpy="0 0 0"/>
-    <mass value="21.681597434756036"/>
-    <inertia ixx="0.129466" iyy="0.073667" izz="0.073667" ixy="0.0" iyz="-0.0" ixz="-0.0"/>
-  </inertial>
-  <visual>
-    <origin xyz="0.195967 0.144669 -0.0289" rpy="0 0 0"/>
+    <origin xyz="-3.6898943472918333e-07 -0.03750028900560054 -3.469446951953614e-18" rpy="0 0 0"/>
+    <mass value="21.681597434756032"/>
+    <inertia ixx="0.073667" iyy="0.129466" izz="0.073667" ixy="0.0" iyz="0.0" ixz="0.0"/>
+  </inertial>
+  <visual>
+    <origin xyz="-0.144669 0.195967 -0.0289" rpy="0 0 0"/>
     <geometry>
       <mesh filename="package://URDF_ROBBOX_description/meshes/wheel_front_right_1.stl" scale="0.001 0.001 0.001"/>
@@ -138,5 +138,5 @@
   </visual>
   <collision>
-    <origin xyz="0.195967 0.144669 -0.0289" rpy="0 0 0"/>
+    <origin xyz="-0.144669 0.195967 -0.0289" rpy="0 0 0"/>
     <geometry>
       <mesh filename="package://URDF_ROBBOX_description/meshes/wheel_front_right_1.stl" scale="0.001 0.001 0.001"/>
@@ -146,10 +146,10 @@
 <link name="wheel_rear_right_1">
   <inertial>
-    <origin xyz="-0.037500000000000006 4.886100667955695e-07 -3.196217084472375e-07" rpy="0 0 0"/>
+    <origin xyz="-4.886100667678139e-07 -0.03750000000000006 -3.196217084333597e-07" rpy="0 0 0"/>
     <mass value="21.68159743475604"/>
-    <inertia ixx="0.129466" iyy="0.073667" izz="0.073667" ixy="0.0" iyz="0.0" ixz="0.0"/>
-  </inertial>
-  <visual>
-    <origin xyz="0.195 -0.143797 -0.028767" rpy="0 0 0"/>
+    <inertia ixx="0.073667" iyy="0.129466" izz="0.073667" ixy="0.0" iyz="0.0" ixz="0.0"/>
+  </inertial>
+  <visual>
+    <origin xyz="0.143797 0.195 -0.028767" rpy="0 0 0"/>
     <geometry>
       <mesh filename="package://URDF_ROBBOX_description/meshes/wheel_rear_right_1.stl" scale="0.001 0.001 0.001"/>
@@ -158,5 +158,5 @@
   </visual>
   <collision>
-    <origin xyz="0.195 -0.143797 -0.028767" rpy="0 0 0"/>
+    <origin xyz="0.143797 0.195 -0.028767" rpy="0 0 0"/>
     <geometry>
       <mesh filename="package://URDF_ROBBOX_description/meshes/wheel_rear_right_1.stl" scale="0.001 0.001 0.001"/>
@@ -165,41 +165,41 @@
 </link>
 <joint name="Rigid 1" type="fixed">
-  <origin xyz="0.065 0.170663 0.4615" rpy="0 0 0"/>
+  <origin xyz="-0.170663 0.065 0.4615" rpy="0 0 0"/>
   <parent link="base_link"/>
   <child link="camera_rpi_1"/>
 </joint>
 <joint name="Rigid 2" type="fixed">
-  <origin xyz="-0.000331 0.170806 0.4765" rpy="0 0 0"/>
+  <origin xyz="-0.170806 -0.000331 0.4765" rpy="0 0 0"/>
   <parent link="base_link"/>
   <child link="lidar_1"/>
 </joint>
 <joint name="Rigid 3" type="fixed">
-  <origin xyz="-0.000238 0.115772 0.4595" rpy="0 0 0"/>
+  <origin xyz="-0.115772 -0.000238 0.4595" rpy="0 0 0"/>
   <parent link="base_link"/>
   <child link="camera_oak_1"/>
 </joint>
 <joint name="Revolute 4" type="continuous">
-  <origin xyz="0.195 0.143797 0.028767" rpy="0 0 0"/>
+  <origin xyz="-0.143797 0.195 0.028767" rpy="0 0 0"/>
   <parent link="base_link"/>
   <child link="wheel_rear_left_1"/>
-  <axis xyz="1.0 0.0 0.0"/>
+  <axis xyz="0.0 1.0 0.0"/>
 </joint>
 <joint name="Revolute 5" type="continuous">
-  <origin xyz="0.195 -0.145731 0.0289" rpy="0 0 0"/>
+  <origin xyz="0.145731 0.195 0.0289" rpy="0 0 0"/>
   <parent link="base_link"/>
   <child link="wheel_front_left_1"/>
-  <axis xyz="1.0 0.0 0.0"/>
+  <axis xyz="0.0 1.0 0.0"/>
 </joint>
 <joint name="Revolute 6" type="continuous">
-  <origin xyz="-0.195967 -0.144669 0.0289" rpy="0 0 0"/>
+  <origin xyz="0.144669 -0.195967 0.0289" rpy="0 0 0"/>
   <parent link="base_link"/>
   <child link="wheel_front_right_1"/>
-  <axis xyz="-1.0 0.0 0.0"/>
+  <axis xyz="0.0 -1.0 0.0"/>
 </joint>
 <joint name="Revolute 7" type="continuous">
-  <origin xyz="-0.195 0.143797 0.028767" rpy="0 0 0"/>
+  <origin xyz="-0.143797 -0.195 0.028767" rpy="0 0 0"/>
   <parent link="base_link"/>
   <child link="wheel_rear_right_1"/>
-  <axis xyz="-1.0 0.0 0.0"/>
+  <axis xyz="0.0 -1.0 0.0"/>
 </joint>
 </robot>
